Commit message: New code architecture
Redution services between Ros-Gazebo from 3 to one.
One service between core-node and controller-node.
One server for 2 clients.

File: last_letter_2/config/param/aircrafts/quadrotor/urdf/model.urdf.xacro (robot description, xacro)
@@ -3,6 +3,5 @@
 <!-- body, airfoil sizes -->
 <xacro:property name="body_s" value="1" />
-<!-- <xacro:property name="pi" value="3.1415" /> -->
-<!-- body link -->
+<!-- body link parameters x, y, z, mass-->
 <xacro:property name="body_x" value="${body_s}" />
 <xacro:property name="body_y" value="${body_s}" />
@@ -22,13 +21,15 @@
         <inertial>
             <mass value="${body_m}" />
-             <inertia ixx="${1/12*body_m*(body_y*body_y+body_z*body_z)}" ixy="0" ixz="0" iyz="0"
-                iyy="${1/12*body_m*(body_x*body_x+body_z*body_z)}" izz="${1/12*body_m*(body_x*body_x+body_y*body_y)}" />
-        </inertial>
-    </link>
+             <inertia   ixx="${1/12*body_m*(body_y*body_y+body_z*body_z)}" ixy="0" ixz="0" iyz="0"
+                        iyy="${1/12*body_m*(body_x*body_x+body_z*body_z)}"
+                        izz="${1/12*body_m*(body_x*body_x+body_y*body_y)}" />
+        </inertial>
+    </link>
+---------------------------------------------------------- 4 quadrotor arms
 <xacro:property name="arm_x" value="${2*body_s}" />
 <xacro:property name="arm_y" value="${0.1*body_s}" />
 <xacro:property name="arm_z" value="${0.1*body_s}" />
 <xacro:property name="arm_m" value="${0.1*body_m}" />
-    <link name="arm_1">
+    <link name="arm1">
         <visual>
         <origin xyz="${arm_x/2} 0 0"/>
@@ -46,14 +47,15 @@
             <origin xyz="${arm_x/2} 0 0"/>
             <mass value="${arm_m}" />
-            <inertia ixx="${1/12*arm_m*(arm_y*arm_y+arm_z*arm_z)}" ixy="0" ixz="0" iyz="0"
-                    iyy="${1/12*arm_m*(arm_x*arm_x+arm_z*arm_z)}" izz="${1/12*arm_m*(arm_x*arm_x+arm_y*arm_y)}" />
-        </inertial>
-    </link>
-    <joint name="body_FLU_to_arm_1" type="fixed">
+            <inertia    ixx="${1/12*arm_m*(arm_y*arm_y+arm_z*arm_z)}" ixy="0" ixz="0" iyz="0"
+                        iyy="${1/12*arm_m*(arm_x*arm_x+arm_z*arm_z)}"
+                        izz="${1/12*arm_m*(arm_x*arm_x+arm_y*arm_y)}" />
+        </inertial>
+    </link>
+    <joint name="body_FLU_to_arm1" type="fixed">
         <origin xyz="${0.9*body_x/2} ${0.9*body_y/2} 0" rpy="0 0 ${pi/4}"/>
         <parent link="body_FLU" />
-        <child link="arm_1" />
-    </joint>
-    <link name="arm_2">
+        <child link="arm1" />
+    </joint>
+    <link name="arm2">
         <visual>
         <origin xyz="${arm_x/2} 0 0"/>
@@ -71,14 +73,15 @@
             <origin xyz="${arm_x/2} 0 0"/>
             <mass value="${arm_m}" />
-            <inertia ixx="${1/12*arm_m*(arm_y*arm_y+arm_z*arm_z)}" ixy="0" ixz="0" iyz="0"
-                iyy="${1/12*arm_m*(arm_x*arm_x+arm_z*arm_z)}" izz="${1/12*arm_m*(arm_x*arm_x+arm_y*arm_y)}" />
-        </inertial>
-    </link>
-    <joint name="body_FLU_to_arm_2" type="fixed">
+            <inertia    ixx="${1/12*arm_m*(arm_y*arm_y+arm_z*arm_z)}" ixy="0" ixz="0" iyz="0"
+                        iyy="${1/12*arm_m*(arm_x*arm_x+arm_z*arm_z)}"
+                        izz="${1/12*arm_m*(arm_x*arm_x+arm_y*arm_y)}" />
+        </inertial>
+    </link>
+    <joint name="body_FLU_to_arm2" type="fixed">
         <origin xyz="-${0.9*body_x/2} ${0.9*body_y/2} 0" rpy="0 0 ${3/4*pi}"/>
         <parent link="body_FLU" />
-        <child link="arm_2" />
-    </joint>
-        <link name="arm_3">
+        <child link="arm2" />
+    </joint>
+        <link name="arm3">
         <visual>
         <origin xyz="${arm_x/2} 0 0"/>
@@ -96,14 +99,15 @@
             <origin xyz="${arm_x/2} 0 0"/>
             <mass value="${arm_m}" />
-            <inertia ixx="${1/12*arm_m*(arm_y*arm_y+arm_z*arm_z)}" ixy="0" ixz="0" iyz="0"
-                iyy="${1/12*arm_m*(arm_x*arm_x+arm_z*arm_z)}" izz="${1/12*arm_m*(arm_x*arm_x+arm_y*arm_y)}" />
-        </inertial>
-    </link>
-    <joint name="body_FLU_to_arm_3" type="fixed">
+            <inertia    ixx="${1/12*arm_m*(arm_y*arm_y+arm_z*arm_z)}" ixy="0" ixz="0" iyz="0"
+                        iyy="${1/12*arm_m*(arm_x*arm_x+arm_z*arm_z)}"
+                        izz="${1/12*arm_m*(arm_x*arm_x+arm_y*arm_y)}" />
+        </inertial>
+    </link>
+    <joint name="body_FLU_to_arm3" type="fixed">
         <origin xyz="-${0.9*body_x/2} -${0.9*body_y/2} 0" rpy="0 0 ${5/4*pi}"/>
         <parent link="body_FLU" />
-        <child link="arm_3" />
-    </joint>
-        <link name="arm_4">
+        <child link="arm3" />
+    </joint>
+        <link name="arm4">
         <visual>
         <origin xyz="${arm_x/2} 0 0"/>
@@ -121,12 +125,13 @@
             <origin xyz="${arm_x/2} 0 0"/>
             <mass value="${arm_m}" />
-            <inertia ixx="${1/12*arm_m*(arm_y*arm_y+arm_z*arm_z)}" ixy="0" ixz="0" iyz="0"
-                iyy="${1/12*arm_m*(arm_x*arm_x+arm_z*arm_z)}" izz="${1/12*arm_m*(arm_x*arm_x+arm_y*arm_y)}" />
-        </inertial>
-    </link>
-    <joint name="body_FLU_to_arm_4" type="fixed">
+            <inertia    ixx="${1/12*arm_m*(arm_y*arm_y+arm_z*arm_z)}" ixy="0" ixz="0" iyz="0"
+                        iyy="${1/12*arm_m*(arm_x*arm_x+arm_z*arm_z)}"
+                        izz="${1/12*arm_m*(arm_x*arm_x+arm_y*arm_y)}" />
+        </inertial>
+    </link>
+    <joint name="body_FLU_to_arm4" type="fixed">
         <origin xyz="${0.9*body_x/2} -${0.9*body_y/2} 0" rpy="0 0 ${7/4*pi}"/>
         <parent link="body_FLU" />
-        <child link="arm_4" />
+        <child link="arm4" />
     </joint>
     ------------------------------------ motors
@@ -135,5 +140,34 @@
 <xacro:property name="motor_z" value="${0.2*body_s}" />
 <xacro:property name="motor_m" value="${0.1*body_m}" />
-     <link name="motor_1">
+<!-- only motor(Number_0f_Motor) acceptable name for motors -->
+     <link name="motor1">
+        <visual>
+        <origin xyz="${motor_x/2} 0 0" rpy="0 0 0"/>
+            <geometry>
+                <box size="${motor_x} ${motor_y} ${motor_z}" />
+            </geometry>
+        </visual>
+        <collision>
+            <origin xyz="${motor_x/2} 0 0" rpy="0 0 0"/>
+            <geometry>
+                <box size="${motor_x} ${motor_y} ${motor_z}" />
+            </geometry>
+        </collision>
+        <inertial>
+            <origin xyz="${motor_x/2} 0 0" rpy="0 0 0"/>
+            <mass value="${motor_m}" />
+            <inertia    ixx="${1/12*motor_m*(motor_y*motor_y+motor_z*motor_z)}" ixy="0" ixz="0" iyz="0"
+                        iyy="${1/12*motor_m*(motor_x*motor_x+motor_z*motor_z)}"
+                        izz="${1/12*motor_m*(motor_x*motor_x+motor_y*motor_y)}" />
+        </inertial>
+    </link>
+    <joint name="arm1_to_motor1" type="revolute">
+        <origin xyz="${arm_x-motor_x/2} 0 ${arm_z/2}" rpy="0 -1.57 0"/>
+        <parent link="arm1" />
+        <child link="motor1" />
+        <!-- <limit lower="-${pi/4}" upper="${pi/4}" effort="10" velocity="3"/> -->
+        <limit effort="1000.0" lower="-0.000872665" upper="0.000872665" velocity="0.5"/>
+    </joint>
+         <link name="motor2">
         <visual>
         <origin xyz="${motor_x/2} 0 0"/>
@@ -151,14 +185,17 @@
             <origin xyz="${motor_x/2} 0 0"/>
             <mass value="${motor_m}" />
-            <inertia ixx="${1/12*motor_m*(motor_y*motor_y+motor_z*motor_z)}" ixy="0" ixz="0" iyz="0"
-                iyy="${1/12*motor_m*(motor_x*motor_x+motor_z*motor_z)}" izz="${1/12*motor_m*(motor_x*motor_x+motor_y*motor_y)}" />
-        </inertial>
-    </link>
-    <joint name="arm_1_to_motor_1" type="continuous">
-        <origin xyz="${arm_x} 0 0" rpy="0 0 0"/>
-        <parent link="arm_1" />
-        <child link="motor_1" />
-    </joint>
-         <link name="motor_2">
+            <inertia    ixx="${1/12*motor_m*(motor_y*motor_y+motor_z*motor_z)}" ixy="0" ixz="0" iyz="0"
+                        iyy="${1/12*motor_m*(motor_x*motor_x+motor_z*motor_z)}"
+                        izz="${1/12*motor_m*(motor_x*motor_x+motor_y*motor_y)}" />
+        </inertial>
+    </link>
+    <joint name="arm2_to_motor2" type="revolute">
+        <origin xyz="${arm_x-motor_x/2} 0 ${arm_z/2}" rpy="0 -1.57 0"/>
+        <parent link="arm2" />
+        <child link="motor2" />
+        <limit effort="1000.0" lower="-0.000872665" upper="0.000872665" velocity="0.5"/>
+        <!-- <limit lower="-${pi/4}" upper="${pi/4}" effort="10" velocity="3"/> -->
+    </joint>
+         <link name="motor3">
         <visual>
         <origin xyz="${motor_x/2} 0 0"/>
@@ -176,14 +213,17 @@
             <origin xyz="${motor_x/2} 0 0"/>
             <mass value="${motor_m}" />
-            <inertia ixx="${1/12*motor_m*(motor_y*motor_y+motor_z*motor_z)}" ixy="0" ixz="0" iyz="0"
-                iyy="${1/12*motor_m*(motor_x*motor_x+motor_z*motor_z)}" izz="${1/12*motor_m*(motor_x*motor_x+motor_y*motor_y)}" />
-        </inertial>
-    </link>
-    <joint name="arm_2_to_motor_2" type="continuous">
-        <origin xyz="${arm_x} 0 0" rpy="0 0 0"/>
-        <parent link="arm_2" />
-        <child link="motor_2" />
-    </joint>
-         <link name="motor_3">
+            <inertia    ixx="${1/12*motor_m*(motor_y*motor_y+motor_z*motor_z)}" ixy="0" ixz="0" iyz="0"
+                        iyy="${1/12*motor_m*(motor_x*motor_x+motor_z*motor_z)}"
+                        izz="${1/12*motor_m*(motor_x*motor_x+motor_y*motor_y)}" />
+        </inertial>
+    </link>
+    <joint name="arm3_to_motor3" type="revolute">
+        <origin xyz="${arm_x-motor_x/2} 0 ${arm_z/2}" rpy="0 -1.57 0"/>
+        <parent link="arm3" />
+        <child link="motor3" />
+        <limit effort="1000.0" lower="-0.000872665" upper="0.000872665" velocity="0.5"/>
+        <!-- <limit lower="-${pi/4}" upper="${pi/4}" effort="10" velocity="3"/> -->
+    </joint>
+    <link name="motor4">
         <visual>
         <origin xyz="${motor_x/2} 0 0"/>
@@ -201,146 +241,128 @@
             <origin xyz="${motor_x/2} 0 0"/>
             <mass value="${motor_m}" />
-            <inertia ixx="${1/12*motor_m*(motor_y*motor_y+motor_z*motor_z)}" ixy="0" ixz="0" iyz="0"
-                iyy="${1/12*motor_m*(motor_x*motor_x+motor_z*motor_z)}" izz="${1/12*motor_m*(motor_x*motor_x+motor_y*motor_y)}" />
-        </inertial>
-    </link>
-    <joint name="arm_3_to_motor_3" type="continuous">
-        <origin xyz="${arm_x} 0 0" rpy="0 0 0"/>
-        <parent link="arm_3" />
-        <child link="motor_3" />
-    </joint>
-    <link name="motor_4">
-        <visual>
-        <origin xyz="${motor_x/2} 0 0"/>
-            <geometry>
-                <box size="${motor_x} ${motor_y} ${motor_z}" />
-            </geometry>
-        </visual>
-        <collision>
-            <origin xyz="${motor_x/2} 0 0"/>
-            <geometry>
-                <box size="${motor_x} ${motor_y} ${motor_z}" />
-            </geometry>
-        </collision>
-        <inertial>
-            <origin xyz="${motor_x/2} 0 0"/>
-            <mass value="${motor_m}" />
-            <inertia ixx="${1/12*motor_m*(motor_y*motor_y+motor_z*motor_z)}" ixy="0" ixz="0" iyz="0"
-                iyy="${1/12*motor_m*(motor_x*motor_x+motor_z*motor_z)}" izz="${1/12*motor_m*(motor_x*motor_x+motor_y*motor_y)}" />
-        </inertial>
-    </link>
-    <joint name="arm_4_to_motor_4" type="continuous">
-        <origin xyz="${arm_x} 0 0" rpy="0 0 0"/>
-        <parent link="arm_4" />
-        <child link="motor_4" />
+            <inertia    ixx="${1/12*motor_m*(motor_y*motor_y+motor_z*motor_z)}" ixy="0" ixz="0" iyz="0"
+                        iyy="${1/12*motor_m*(motor_x*motor_x+motor_z*motor_z)}"
+                        izz="${1/12*motor_m*(motor_x*motor_x+motor_y*motor_y)}" />
+        </inertial>
+    </link>
+    <joint name="arm4_to_motor4" type="revolute">
+        <origin xyz="${arm_x-motor_x/2} 0 ${arm_z/2}" rpy="0 -1.57 0"/>
+        <parent link="arm4" />
+        <child link="motor4" />
+        <limit effort="1000.0" lower="-0.000872665" upper="0.000872665" velocity="0.5"/>
+        <!-- <limit lower="-${pi/4}" upper="${pi/4}" effort="10" velocity="3"/> -->
     </joint>
  ------------------------------------- propellers
 <!-- arm link -->
-<xacro:property name="prop_arm_m" value="${body_m/20}" />
-<xacro:property name="prop_arm_r" value="${body_s/40}" />
-<xacro:property name="prop_arm_h" value="${body_s/40}" />
-    <link name="prop_arm_1">
-        <visual>
-            <origin xyz="0 0 ${prop_arm_h/2}" rpy="0 0 0"/>
-            <geometry>
-                <cylinder radius="${prop_arm_r}" length="${prop_arm_h}" />
-            </geometry>
-        </visual>
-        <collision>
-            <origin xyz="0 0 ${prop_arm_h/2}" rpy="0 0 0"/>
-            <geometry>
-                <cylinder radius="${prop_arm_r}" length="${prop_arm_h}" />
-            </geometry>
-        </collision>
-        <inertial>
-            <origin xyz="0 0 ${prop_arm_h/2}" />
-            <mass value="${prop_arm_m}" />
-            <inertia ixx="${1/12*prop_arm_m*prop_arm_h*prop_arm_h+1/4*prop_arm_m*prop_arm_r*prop_arm_r}" ixy="0" ixz="0" iyz="0"
-                iyy="${1/12*prop_arm_m*prop_arm_h*prop_arm_h+1/4*prop_arm_m*prop_arm_r*prop_arm_r}" izz="${1/2*prop_arm_m*prop_arm_r*prop_arm_r}" />
-        </inertial>
-    </link>
-    <joint name="motor_1_to_prop_arm_1" type="continuous">
-        <origin xyz="${motor_x/2} 0 ${motor_z/2}" rpy="0 0 0" />
-        <axis xyz="0 0 1" />
-        <parent link="motor_1" />
-        <child link="prop_arm_1" />
-    </joint>
-        <link name="prop_arm_2">
-        <visual>
-            <origin xyz="0 0 ${prop_arm_h/2}" rpy="0 0 0"/>
-            <geometry>
-                <cylinder radius="${prop_arm_r}" length="${prop_arm_h}" />
-            </geometry>
-        </visual>
-        <collision>
-            <origin xyz="0 0 ${prop_arm_h/2}" rpy="0 0 0"/>
-            <geometry>
-                <cylinder radius="${prop_arm_r}" length="${prop_arm_h}" />
-            </geometry>
-        </collision>
-        <inertial>
-            <origin xyz="0 0 ${prop_arm_h/2}" />
-            <mass value="${prop_arm_m}" />
-            <inertia ixx="${1/12*prop_arm_m*prop_arm_h*prop_arm_h+1/4*prop_arm_m*prop_arm_r*prop_arm_r}" ixy="0" ixz="0" iyz="0"
-                iyy="${1/12*prop_arm_m*prop_arm_h*prop_arm_h+1/4*prop_arm_m*prop_arm_r*prop_arm_r}" izz="${1/2*prop_arm_m*prop_arm_r*prop_arm_r}" />
-        </inertial>
-    </link>
-    <joint name="motor_2_to_prop_arm_2" type="continuous">
-        <origin xyz="${motor_x/2} 0 ${motor_z/2}" rpy="0 0 0" />
-        <axis xyz="0 0 1" />
-        <parent link="motor_2" />
-        <child link="prop_arm_2" />
-    </joint>
-        <link name="prop_arm_3">
-        <visual>
-            <origin xyz="0 0 ${prop_arm_h/2}" rpy="0 0 0"/>
-            <geometry>
-                <cylinder radius="${prop_arm_r}" length="${prop_arm_h}" />
-            </geometry>
-        </visual>
-        <collision>
-            <origin xyz="0 0 ${prop_arm_h/2}" rpy="0 0 0"/>
-            <geometry>
-                <cylinder radius="${prop_arm_r}" length="${prop_arm_h}" />
-            </geometry>
-        </collision>
-        <inertial>
-            <origin xyz="0 0 ${prop_arm_h/2}" />
-            <mass value="${prop_arm_m}" />
-            <inertia ixx="${1/12*prop_arm_m*prop_arm_h*prop_arm_h+1/4*prop_arm_m*prop_arm_r*prop_arm_r}" ixy="0" ixz="0" iyz="0"
-                iyy="${1/12*prop_arm_m*prop_arm_h*prop_arm_h+1/4*prop_arm_m*prop_arm_r*prop_arm_r}" izz="${1/2*prop_arm_m*prop_arm_r*prop_arm_r}" />
-        </inertial>
-    </link>
-    <joint name="motor_3_to_prop_arm_3" type="continuous">
-        <origin xyz="${motor_x/2} 0 ${motor_z/2}" rpy="0 0 0" />
-        <axis xyz="0 0 1" />
-        <parent link="motor_3" />
-        <child link="prop_arm_3" />
-    </joint>
-        <link name="prop_arm_4">
-        <visual>
-            <origin xyz="0 0 ${prop_arm_h/2}" rpy="0 0 0"/>
-            <geometry>
-                <cylinder radius="${prop_arm_r}" length="${prop_arm_h}" />
-            </geometry>
-        </visual>
-        <collision>
-            <origin xyz="0 0 ${prop_arm_h/2}" rpy="0 0 0"/>
-            <geometry>
-                <cylinder radius="${prop_arm_r}" length="${prop_arm_h}" />
-            </geometry>
-        </collision>
-        <inertial>
-            <origin xyz="0 0 ${prop_arm_h/2}" />
-            <mass value="${prop_arm_m}" />
-            <inertia ixx="${1/12*prop_arm_m*prop_arm_h*prop_arm_h+1/4*prop_arm_m*prop_arm_r*prop_arm_r}" ixy="0" ixz="0" iyz="0"
-                iyy="${1/12*prop_arm_m*prop_arm_h*prop_arm_h+1/4*prop_arm_m*prop_arm_r*prop_arm_r}" izz="${1/2*prop_arm_m*prop_arm_r*prop_arm_r}" />
-        </inertial>
-    </link>
-    <joint name="motor_4_to_prop_arm_4" type="continuous">
-        <origin xyz="${motor_x/2} 0 ${motor_z/2}" rpy="0 0 0" />
-        <axis xyz="0 0 1" />
-        <parent link="motor_4" />
-        <child link="prop_arm_4" />
+<xacro:property name="axle_m" value="${body_m/20}" />
+<xacro:property name="axle_r" value="${body_s/40}" />
+<xacro:property name="axle_h" value="${body_s/40}" />
+    <link name="axle1">
+        <visual>
+            <origin xyz="${axle_h/2} 0 0" rpy="0 ${pi/2} 0"/>
+            <geometry>
+                <cylinder radius="${axle_r}" length="${axle_h}" />
+            </geometry>
+        </visual>
+        <collision>
+            <origin xyz="${axle_h/2} 0 0" rpy="0 ${pi/2} 0"/>
+            <geometry>
+                <cylinder radius="${axle_r}" length="${axle_h}" />
+            </geometry>
+        </collision>
+        <inertial>
+            <origin xyz="${axle_h/2} 0 0" />
+            <mass value="${axle_m}" />
+            <inertia    ixx="${1/12*axle_m*axle_h*axle_h+1/4*axle_m*axle_r*axle_r}" ixy="0" ixz="0" iyz="0"
+                        iyy="${1/12*axle_m*axle_h*axle_h+1/4*axle_m*axle_r*axle_r}"
+                        izz="${1/2*axle_m*axle_r*axle_r}" />
+        </inertial>
+    </link>
+    <joint name="motor1_to_axle1" type="continuous">
+        <origin xyz="${motor_x} 0 0" rpy="0 0 0"/>
+        <axis xyz="1 0 0" />
+        <parent link="motor1" />
+        <child link="axle1" />
+    </joint>
+        <link name="axle2">
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
Commit message: Remove details
Remove some code useless lines

File: last_letter_2/config/param/aircrafts/csl_2k19/urdf/model.urdf.xacro (robot description, xacro)
@@ -10,5 +10,5 @@
 <xacro:property name="body_h" value="${2.5*body_s}" />
 <xacro:property name="body_r" value="${0.5*body_s}" />
-<xacro:property name="body_m" value="${body_s/10}" />
+<xacro:property name="body_m" value="${0.3*mass}" />
     <!-- only body_FLU acceptable name for base_link -->
     <link name="body_FLU">
@@ -38,5 +38,5 @@
 <xacro:property name="airfoil_y" value="${airfoil_s*6}" />
 <xacro:property name="airfoil_z" value="${airfoil_s/10}"/>
-<xacro:property name="airfoil_m" value="2" />               ----airfoil mass
+<xacro:property name="airfoil_m" value="${0.3*mass}" />               ----airfoil mass
     <!-- only airfoil(Number_0f_Airfoil) acceptable name for airfoils -->
     <link name="airfoil1">
@@ -70,5 +70,5 @@
 <xacro:property name="motor_y" value="${body_s/5}" />
 <xacro:property name="motor_z" value="${body_s/5}" />
-<xacro:property name="motor_m" value="${body_m/5}" />
+<xacro:property name="motor_m" value="${0.3*mass}" />
 <!-- only motor(Number_0f_Motor) acceptable name for motors -->
  <link name="motor1">
@@ -103,5 +103,5 @@
 <xacro:property name="axle_h" value="${body_h/12}" />
 <xacro:property name="axle_r" value="${body_r/10}" />
-<xacro:property name="axle_m" value="${body_m/2}" />
+<xacro:property name="axle_m" value="${0.005*mass}" />
     <link name="axle1">
         <visual>
@@ -135,5 +135,5 @@
 <xacro:property name="propeller_y" value="${0.2*body_s}" />
 <xacro:property name="propeller_z" value="${0.05*body_s}" />
-<xacro:property name="propeller_m" value="${body_m/2}" />
+<xacro:property name="propeller_m" value="${0.015*mass}" />
     <link name="propeller1">
         <visual>
@@ -164,5 +164,5 @@
 <xacro:property name="wheel_base_y" value="${2*body_s}" />
 <xacro:property name="wheel_base_z" value="${0.05*body_s}" />
-<xacro:property name="wheel_base_m" value="${0.5*body_m}" />
+<xacro:property name="wheel_base_m" value="${0.05*mass}" />
     <link name="wheel_base">
         <visual>
@@ -191,5 +191,5 @@
 <xacro:property name="left_wheel_r" value="${0.3*body_s}" />
 <xacro:property name="left_wheel_h" value="${0.1*body_s}" />
-<xacro:property name="left_wheel_m" value="${body_m/2}" />
+<xacro:property name="left_wheel_m" value="${0.01*mass}" />
     <link name="left_wheel">
         <visual>
@@ -253,5 +253,5 @@
 <!-- rear wheel link parameters, rad, mass -->
 <xacro:property name="rear_wheel_m" value="${body_m/2}" />
-<xacro:property name="rear_wheel_r" value="${0.1*body_s}" />
+<xacro:property name="rear_wheel_r" value="${0.01*mass}" />
     <link name="rear_wheel">
         <visual>
