Commit message: 3-wing plane model
A plane with 3 wings, one for each move of roll pitch yaw.

File: last_letter_2/config/param/aircrafts/csl_2k21/urdf/model.urdf.xacro (robot description, xacro)
@@ -1,4 +1,4 @@
 <?xml version="1.0"?>
-<robot name="cassna 172" xmlns:xacro="http://www.ros.org/wiki/xacro">
+<robot name="plane" xmlns:xacro="http://www.ros.org/wiki/xacro">
 <xacro:property name="source" value="$(find last_letter_2)/config/param/aircrafts/csl_2k19/rigidBody.yaml" />
 <xacro:property name="dictionary" value="${load_yaml(source)}"/>
@@ -7,9 +7,8 @@
 <xacro:property name="body_s" value="1" />
 <xacro:property name="airfoil_s" value="1" />
-<xacro:property name="whole_mass" value="100" />
 <!-- body link , body_height, body_rad, body_mass -->
-<xacro:property name="body_h" value="${8.28*body_s}" />
-<xacro:property name="body_r" value="${0.8*body_s}" />
-<xacro:property name="body_m" value="${0.4*whole_mass}" />
+<xacro:property name="body_h" value="${2.5*body_s}" />
+<xacro:property name="body_r" value="${0.5*body_s}" />
+<xacro:property name="body_m" value="${0.3*mass}" />
     <!-- only body_FLU acceptable name for base_link -->
     <link name="body_FLU">
@@ -36,38 +35,67 @@
     ----------------------------------------------------------------------------  airfoils
 <!-- airfoil1 link parameters , x, y, z, mass-->
-<xacro:property name="airfoil1_x" value="${2*body_s}" />
-<xacro:property name="airfoil1_y" value="${11*body_s}" />
-<xacro:property name="airfoil1_z" value="${body_s/5}"/>
-<xacro:property name="airfoil1_m" value="${0.3*whole_mass}" />               ----airfoil1 mass
+<xacro:property name="airfoil_x" value="${airfoil_s/2}" />
+<xacro:property name="airfoil_y" value="${airfoil_s*6}" />
+<xacro:property name="airfoil_z" value="${airfoil_s/10}"/>
+<xacro:property name="airfoil_m" value="${0.3*mass}" />               ----airfoil mass
     <!-- only airfoil(Number_0f_Airfoil) acceptable name for airfoils -->
     <link name="airfoil1">
         <visual>
             <geometry>
-                <box size="${airfoil1_x} ${airfoil1_y} ${airfoil1_z}" />
-            </geometry>
-        </visual>
-        <collision>
-            <geometry>
-                <box size="${airfoil1_x} ${airfoil1_y} ${airfoil1_z}" />
+                <box size="${airfoil_x} ${airfoil_y} ${airfoil_z}" />
+            </geometry>
+        </visual>
+        <collision>
+            <geometry>
+                <box size="${airfoil_x} ${airfoil_y} ${airfoil_z}" />
             </geometry>
         </collision>
          <inertial>
-            <mass value="${airfoil1_m}" />
-            <inertia    ixx="${1/12*airfoil1_m*(airfoil1_y*airfoil1_y+airfoil1_z*airfoil1_z)}" ixy="0" ixz="0" iyz="0"
-                        iyy="${1/12*airfoil1_m*(airfoil1_x*airfoil1_x+airfoil1_z*airfoil1_z)}"
-                        izz="${1/12*airfoil1_m*(airfoil1_x*airfoil1_x+airfoil1_y*airfoil1_y)}" />
+            <mass value="${airfoil_m}" />
+            <inertia    ixx="${1/12*airfoil_m*(airfoil_y*airfoil_y+airfoil_z*airfoil_z)}" ixy="0" ixz="0" iyz="0"
+                        iyy="${1/12*airfoil_m*(airfoil_x*airfoil_x+airfoil_z*airfoil_z)}"
+                        izz="${1/12*airfoil_m*(airfoil_x*airfoil_x+airfoil_y*airfoil_y)}" />
         </inertial>
     </link>
     <joint name="body_FLU_to_airfoil1" type="revolute">
-        <origin xyz="${body_h/6} 0 ${body_r-airfoil1_z/2}" rpy ="0 0 0"/>
+        <origin xyz="${body_h/15} 0 ${body_r-airfoil_z/2}" rpy ="0 0 0"/>
         <parent link="body_FLU" />
         <child link="airfoil1" />
         <limit effort="1000.0" velocity="0.5"/>   ---default limits upper=lower=0
     </joint>
-<!-- airfoil2 link parameters , x, y, z, mass-->
-<xacro:property name="airfoil2_x" value="${body_s}" />
-<xacro:property name="airfoil2_y" value="${3.4*body_s}" />
-<xacro:property name="airfoil2_z" value="${body_s/5}"/>
-<xacro:property name="airfoil2_m" value="${0.1*whole_mass}" />               ----airfoil2 mass
+    ----------------------------------------------------------------------------------- motors
+<!-- motor link -->
+<!-- motor parameters , x, y, z, mass -->
+<xacro:property name="motor_x" value="${body_s/10}" />
+<xacro:property name="motor_y" value="${body_s/5}" />
+<xacro:property name="motor_z" value="${body_s/5}" />
+<xacro:property name="motor_m" value="${0.3*mass}" />
+<!-- only motor(Number_0f_Motor) acceptable name for motors -->
+ <link name="motor1">
+        <visual>
+            <origin xyz="${0.5*motor_x} 0 0"/>
+            <geometry>
+                <box size="${motor_x} ${motor_y} ${motor_z}" />
+            </geometry>
+        </visual>
+        <collision>
+            <origin xyz="${0.5*motor_x} 0 0"/>
+            <geometry>
+                <box size="${motor_x} ${motor_y} ${motor_z}" />
+            </geometry>
+        </collision>
+        <inertial>
+            <origin xyz="${0.5*motor_x} 0 0"/>
+            <mass value="${motor_m}" />
+            <inertia    ixx="${1/12*motor_m*(motor_y*motor_y+motor_z*motor_z)}" ixy="0" ixz="0" iyz="0"
+                        iyy="${1/12*motor_m*(motor_x*motor_x+motor_z*motor_z)}"
+                        izz="${1/12*motor_m*(motor_x*motor_x+motor_y*motor_y)}" />
+        </inertial>
+    </link>
+ <!-- airfoil2 link parameters , x, y, z, mass-->
+<xacro:property name="airfoil2_x" value="${0.3*body_s}" />
+<xacro:property name="airfoil2_y" value="${2*body_s}" />
+<xacro:property name="airfoil2_z" value="${0.1*body_s}"/>
+<xacro:property name="airfoil2_m" value="${0.01*mass}" />               ----airfoil2 mass
     <!-- only airfoil(Number_0f_Airfoil) acceptable name for airfoils -->
     <link name="airfoil2">
@@ -96,8 +124,8 @@
     </joint>
 <!-- airfoil3 link parameters , x, y, z, mass-->
-<xacro:property name="airfoil3_x" value="${body_s}" />
-<xacro:property name="airfoil3_y" value="${2*body_s}" />
-<xacro:property name="airfoil3_z" value="${body_s/5}"/>
-<xacro:property name="airfoil3_m" value="${0.1*whole_mass}" />               ----airfoil3 mass
+<xacro:property name="airfoil3_x" value="${0.3*body_s}" />
+<xacro:property name="airfoil3_y" value="${0.5*body_s}" />
+<xacro:property name="airfoil3_z" value="${0.1*body_s}"/>
+<xacro:property name="airfoil3_m" value="${0.01*mass}" />               ----airfoil3 mass
     <!-- only airfoil(Number_0f_Airfoil) acceptable name for airfoils -->
     <link name="airfoil3">
@@ -120,38 +148,9 @@
     </link>
     <joint name="body_FLU_to_airfoil3" type="revolute">
-        <origin xyz="${-body_h/2+airfoil3_x/2} 0 ${airfoil3_y/2}" rpy ="${pi/2} 0 0"/>
+        <origin xyz="${-body_h/2+airfoil3_x/2} 0 ${body_r+airfoil3_y/2}" rpy ="1.57 0 0"/>
         <parent link="body_FLU" />
         <child link="airfoil3" />
         <limit effort="1000.0" velocity="0.5"/>   ---default limits upper=lower=0
     </joint>
-    ----------------------------------------------------------------------------------- motors
-<!-- motor1 link -->
-<!-- motor1 parameters , x, y, z, mass -->
-<xacro:property name="motor1_x" value="${body_s/10}" />
-<xacro:property name="motor1_y" value="${body_s/5}" />
-<xacro:property name="motor1_z" value="${body_s/5}" />
-<xacro:property name="motor1_m" value="${whole_mass/100}" />
-<!-- only motor1(Number_0f_Motor1) acceptable name for motor1s -->
- <link name="motor1">
-        <visual>
-            <origin xyz="${0.5*motor1_x} 0 0"/>
-            <geometry>
-                <box size="${motor1_x} ${motor1_y} ${motor1_z}" />
-            </geometry>
-        </visual>
-        <collision>
-            <origin xyz="${0.5*motor1_x} 0 0"/>
-            <geometry>
-                <box size="${motor1_x} ${motor1_y} ${motor1_z}" />
-            </geometry>
-        </collision>
-        <inertial>
-            <origin xyz="${0.5*motor1_x} 0 0"/>
-            <mass value="${motor1_m}" />
-            <inertia    ixx="${1/12*motor1_m*(motor1_y*motor1_y+motor1_z*motor1_z)}" ixy="0" ixz="0" iyz="0"
-                        iyy="${1/12*motor1_m*(motor1_x*motor1_x+motor1_z*motor1_z)}"
-                        izz="${1/12*motor1_m*(motor1_x*motor1_x+motor1_y*motor1_y)}" />
-        </inertial>
-    </link>
     <joint name="body_FLU_to_motor1" type="revolute">
         <origin xyz="${0.5*body_h} 0 0" rpy="0 0 0" />
@@ -162,7 +161,7 @@
  -----------------------------------------------------------------------------------propeller
 <!-- axle link parameters height, rad, mass-->
-<xacro:property name="axle_h" value="${body_h/100}" />
+<xacro:property name="axle_h" value="${body_h/12}" />
 <xacro:property name="axle_r" value="${body_r/10}" />
-<xacro:property name="axle_m" value="${body_m/100}" />
+<xacro:property name="axle_m" value="${0.005*mass}" />
     <link name="axle1">
         <visual>
@@ -187,5 +186,5 @@
     </link>
     <joint name="motor1_to_axle1" type="continuous">
-        <origin xyz="${motor1_x} 0 0" rpy="0 0 0" />
+        <origin xyz="${motor_x} 0 0" rpy="0 0 0" />
         <axis xyz="1 0 0" />
         <parent link="motor1" />
@@ -193,8 +192,8 @@
     </joint>
 <!-- propeller link parameters x, y, z, mass -->
-<xacro:property name="propeller_x" value="${1.8*body_s}" />
+<xacro:property name="propeller_x" value="${0.8*body_s}" />
 <xacro:property name="propeller_y" value="${0.2*body_s}" />
 <xacro:property name="propeller_z" value="${0.05*body_s}" />
-<xacro:property name="propeller_m" value="${body_m/100}" />
+<xacro:property name="propeller_m" value="${0.015*mass}" />
     <link name="propeller1">
         <visual>
@@ -223,7 +222,7 @@
      <!-- wheel_base_link parameters, x, y, z, mass-->
 <xacro:property name="wheel_base_x" value="${0.05*body_s}" />
-<xacro:property name="wheel_base_y" value="${4*body_s}" />
+<xacro:property name="wheel_base_y" value="${2*body_s}" />
 <xacro:property name="wheel_base_z" value="${0.05*body_s}" />
-<xacro:property name="wheel_base_m" value="${body_m/100}" />
+<xacro:property name="wheel_base_m" value="${0.05*mass}" />
     <link name="wheel_base">
         <visual>
@@ -252,5 +251,5 @@
 <xacro:property name="left_wheel_r" value="${0.3*body_s}" />
 <xacro:property name="left_wheel_h" value="${0.1*body_s}" />
-<xacro:property name="left_wheel_m" value="${body_m/100}" />
+<xacro:property name="left_wheel_m" value="${0.01*mass}" />
     <link name="left_wheel">
         <visual>
@@ -283,5 +282,5 @@
 <xacro:property name="right_wheel_r" value="${left_wheel_r}" />
 <xacro:property name="right_wheel_h" value="${left_wheel_h}" />
-<xacro:property name="right_wheel_m" value="${whole_mass/100}" />
+<xacro:property name="right_wheel_m" value="${left_wheel_m}" />
     <link name="right_wheel">
         <visual>
@@ -313,6 +312,6 @@
     ------------------------------------------------------------------------------------ rear sphere wheel
 <!-- rear wheel link parameters, rad, mass -->
-<xacro:property name="rear_wheel_m" value="${whole_mass/100}" />
-<xacro:property name="rear_wheel_r" value="${0.1*body_s}" />
+<xacro:property name="rear_wheel_m" value="${body_m/2}" />
+<xacro:property name="rear_wheel_r" value="${0.01*mass}" />
     <link name="rear_wheel">
         <visual>
@@ -343,5 +342,5 @@
     <plugin name="model_plugin" filename="libmodel_plugin.so"/>
     <plugin name="joint_state_publisher" filename="libgazebo_ros_joint_state_publisher.so">
-        <jointName>body_FLU_to_airfoil1,body_FLU_to_airfoil2,body_FLU_to_airfoil3, body_FLU_to_motor1, wheel_base_to_left_wheel, wheel_base_to_right_wheel, body_FLU_to_rear_wheel </jointName>
+        <jointName>body_FLU_to_airfoil1,body_FLU_to_airfoil2,body_FLU_to_airfoil3, body_FLU_to_motor1, motor1_to_axle1, wheel_base_to_left_wheel, wheel_base_to_right_wheel, body_FLU_to_rear_wheel </jointName>
         <robotNamespace>last_letter_2</robotNamespace>
         <updateRate>0</updateRate>
