Commit message: Controller_set_up
Make controller node subscribe on model_states and take into account the model_states in calculation of controller Inputs.

File: last_letter_2/config/param/aircrafts/quadrotor/urdf/model.urdf.xacro (robot description, xacro)
@@ -1,4 +1,7 @@
 <?xml version="1.0"?>
 <robot name="quadrotor" xmlns:xacro="http://www.ros.org/wiki/xacro">
+<xacro:property name="source" value="$(find last_letter_2)/config/param/aircrafts/quadrotor/rigidBody.yaml" />
+<xacro:property name="dictionary" value="${load_yaml(source)}"/>
+<xacro:property name="body_mass" value="${dictionary['airframe/m']}"/>
 <!-- body, airfoil sizes -->
 <xacro:property name="body_s" value="1" />
@@ -7,5 +10,5 @@
 <xacro:property name="body_y" value="${body_s}" />
 <xacro:property name="body_z" value="${body_s/5}" />
-<xacro:property name="body_m" value="2" />
+<xacro:property name="body_m" value="${body_mass}" />
     <link name="body_FLU">
         <visual>
@@ -53,5 +56,5 @@
     </link>
     <joint name="body_FLU_to_arm1" type="fixed">
-        <origin xyz="${0.9*body_x/2} ${0.9*body_y/2} 0" rpy="0 0 ${pi/4}"/>
+        <origin xyz="${0.9*body_x/2} -${0.9*body_y/2} 0" rpy="0 0 ${7/4*pi}"/>
         <parent link="body_FLU" />
         <child link="arm1" />
@@ -79,5 +82,5 @@
     </link>
     <joint name="body_FLU_to_arm2" type="fixed">
-        <origin xyz="-${0.9*body_x/2} ${0.9*body_y/2} 0" rpy="0 0 ${3/4*pi}"/>
+        <origin xyz="-${0.9*body_x/2} -${0.9*body_y/2} 0" rpy="0 0 ${5/4*pi}"/>
         <parent link="body_FLU" />
         <child link="arm2" />
@@ -105,5 +108,5 @@
     </link>
     <joint name="body_FLU_to_arm3" type="fixed">
-        <origin xyz="-${0.9*body_x/2} -${0.9*body_y/2} 0" rpy="0 0 ${5/4*pi}"/>
+        <origin xyz="-${0.9*body_x/2} ${0.9*body_y/2} 0" rpy="0 0 ${3/4*pi}"/>
         <parent link="body_FLU" />
         <child link="arm3" />
@@ -131,5 +134,5 @@
     </link>
     <joint name="body_FLU_to_arm4" type="fixed">
-        <origin xyz="${0.9*body_x/2} -${0.9*body_y/2} 0" rpy="0 0 ${7/4*pi}"/>
+        <origin xyz="${0.9*body_x/2} ${0.9*body_y/2} 0" rpy="0 0 ${1/4*pi}"/>
         <parent link="body_FLU" />
         <child link="arm4" />

Commit message: PD drone controller
Stabilize and altitude PD controller for multirotor

File: last_letter_2/config/param/aircrafts/quadrotor/urdf/model.urdf.xacro (robot description, xacro)
@@ -13,4 +13,5 @@
     <link name="body_FLU">
         <visual>
+        <origin rpy="0 0 0.785"/>
             <geometry>
                <box size="${body_x} ${body_y} ${body_z}" />
@@ -18,4 +19,5 @@
         </visual>
         <collision>
+        <origin rpy="0 0 0.785"/>
             <geometry>
                <box size="${body_x} ${body_y} ${body_z}" />
@@ -23,4 +25,5 @@
         </collision>
         <inertial>
+        <origin rpy="0 0 0.785"/>
             <mass value="${body_m}" />
              <inertia   ixx="${1/12*body_m*(body_y*body_y+body_z*body_z)}" ixy="0" ixz="0" iyz="0"
@@ -56,5 +59,5 @@
     </link>
     <joint name="body_FLU_to_arm1" type="fixed">
-        <origin xyz="${0.9*body_x/2} -${0.9*body_y/2} 0" rpy="0 0 ${7/4*pi}"/>
+        <origin xyz="${0.9*body_x/2} 0 0" rpy="0 0 0"/>
         <parent link="body_FLU" />
         <child link="arm1" />
@@ -82,5 +85,5 @@
     </link>
     <joint name="body_FLU_to_arm2" type="fixed">
-        <origin xyz="-${0.9*body_x/2} -${0.9*body_y/2} 0" rpy="0 0 ${5/4*pi}"/>
+        <origin xyz="0 -${0.9*body_y/2} 0" rpy="0 0 ${3/2*pi}"/>
         <parent link="body_FLU" />
         <child link="arm2" />
@@ -108,5 +111,5 @@
     </link>
     <joint name="body_FLU_to_arm3" type="fixed">
-        <origin xyz="-${0.9*body_x/2} ${0.9*body_y/2} 0" rpy="0 0 ${3/4*pi}"/>
+        <origin xyz="-${0.9*body_x/2} 0 0" rpy="0 0 ${pi}"/>
         <parent link="body_FLU" />
         <child link="arm3" />
@@ -134,5 +137,5 @@
     </link>
     <joint name="body_FLU_to_arm4" type="fixed">
-        <origin xyz="${0.9*body_x/2} ${0.9*body_y/2} 0" rpy="0 0 ${1/4*pi}"/>
+        <origin xyz="0 ${0.9*body_y/2} 0" rpy="0 0 ${1/2*pi}"/>
         <parent link="body_FLU" />
         <child link="arm4" />

Commit message: Propeller Rotation (Omega)
Make propellers spin, relative to input signals

File: last_letter_2/config/param/aircrafts/quadrotor/urdf/model.urdf.xacro (robot description, xacro)
@@ -366,5 +366,5 @@
         </inertial>
     </link>
-    <joint name="motor_4_to_axle4" type="continuous">
+    <joint name="motor4_to_axle4" type="continuous">
         <origin xyz="${motor_x} 0 0" rpy="0 0 0"/>
         <axis xyz="1 0 0" />
@@ -489,5 +489,5 @@
     <plugin name="model_plugin" filename="libmodel_plugin.so"/>
     <plugin name="joint_state_publisher" filename="libgazebo_ros_joint_state_publisher.so">
-        <jointName>arm1_to_motor1, arm2_to_motor2, arm3_to_motor3,arm4_to_motor4,motor1_to_axle1,motor2_to_axle2,motor3_to_axle3,motor_4_to_axle4 </jointName>
+        <jointName>arm1_to_motor1, arm2_to_motor2, arm3_to_motor3,arm4_to_motor4,motor1_to_axle1,motor2_to_axle2,motor3_to_axle3,motor4_to_axle4 </jointName>
         <robotNamespace>last_letter_2</robotNamespace>
         <updateRate>0</updateRate>
