Commit message: Code small changes
Change some names of variables, add some files and delete others.

File: last_letter_2/config/param/aircrafts/plane_1wing/urdf/model.urdf.xacro (robot description, xacro)
@@ -1,5 +1,5 @@
 <?xml version="1.0"?>
 <robot name="plane" xmlns:xacro="http://www.ros.org/wiki/xacro">
-<xacro:property name="source" value="$(find last_letter_2)/config/param/aircrafts/csl_2k19/rigidBody.yaml" />
+<xacro:property name="source" value="$(find last_letter_2)/config/param/aircrafts/plane_1wing/rigidBody.yaml" />
 <xacro:property name="dictionary" value="${load_yaml(source)}"/>
 <xacro:property name="mass" value="${dictionary['airframe/m']}"/>

File: last_letter_2/config/param/aircrafts/plane_3wing/urdf/model.urdf.xacro (robot description, xacro)
@@ -1,5 +1,5 @@
 <?xml version="1.0"?>
 <robot name="plane" xmlns:xacro="http://www.ros.org/wiki/xacro">
-<xacro:property name="source" value="$(find last_letter_2)/config/param/aircrafts/csl_2k19/rigidBody.yaml" />
+<xacro:property name="source" value="$(find last_letter_2)/config/param/aircrafts/plane_3wing/rigidBody.yaml" />
 <xacro:property name="dictionary" value="${load_yaml(source)}"/>
 <xacro:property name="mass" value="${dictionary['airframe/m']}"/>
