Commit message: Hexacopter
Add Hexacopter model. Clear environment.cpp file. Change some variable names

File: last_letter_2/config/param/aircrafts/quadcopter/urdf/model.urdf.xacro (robot description, xacro)
@@ -1,5 +1,5 @@
 <?xml version="1.0"?>
-<robot name="quadrotor" xmlns:xacro="http://www.ros.org/wiki/xacro">
-<xacro:property name="source" value="$(find last_letter_2)/config/param/aircrafts/quadrotor/rigidBody.yaml" />
+<robot name="quadcopter" xmlns:xacro="http://www.ros.org/wiki/xacro">
+<xacro:property name="source" value="$(find last_letter_2)/config/param/aircrafts/quadcopter/rigidBody.yaml" />
 <xacro:property name="dictionary" value="${load_yaml(source)}"/>
 <xacro:property name="body_mass" value="${dictionary['airframe/m']}"/>
@@ -32,5 +32,5 @@
         </inertial>
     </link>
----------------------------------------------------------- 4 quadrotor arms
+---------------------------------------------------------- 4 quadcopter arms
 <xacro:property name="arm_x" value="${2*body_s}" />
 <xacro:property name="arm_y" value="${0.1*body_s}" />
