Commit message: Useless code clean
Clean the code from useless lines

File: last_letter_2/config/param/aircrafts/hexacopter/urdf/model.urdf.xacro (robot description, xacro)
@@ -1,5 +1,5 @@
 <?xml version="1.0"?>
 <robot name="hexacopter" xmlns:xacro="http://www.ros.org/wiki/xacro">
-<xacro:property name="source" value="$(find last_letter_2)/config/param/aircrafts/hexacopter/rigidBody.yaml" />
+<xacro:property name="source" value="$(find last_letter_2)/config/param/aircrafts/hexacopter/mass.yaml" />
 <xacro:property name="dictionary" value="${load_yaml(source)}"/>
 <xacro:property name="body_mass" value="${dictionary['airframe/m']}"/>

File: last_letter_2/config/param/aircrafts/plane_1wing/urdf/model.urdf.xacro (robot description, xacro)
@@ -1,5 +1,5 @@
 <?xml version="1.0"?>
 <robot name="plane" xmlns:xacro="http://www.ros.org/wiki/xacro">
-<xacro:property name="source" value="$(find last_letter_2)/config/param/aircrafts/plane_1wing/rigidBody.yaml" />
+<xacro:property name="source" value="$(find last_letter_2)/config/param/aircrafts/plane_1wing/mass.yaml" />
 <xacro:property name="dictionary" value="${load_yaml(source)}"/>
 <xacro:property name="mass" value="${dictionary['airframe/m']}"/>

File: last_letter_2/config/param/aircrafts/plane_1wing_sensors/urdf/model.urdf.xacro (robot description, xacro)
@@ -1,5 +1,5 @@
 <?xml version="1.0"?>
 <robot name="plane_sensors" xmlns:xacro="http://www.ros.org/wiki/xacro">
-<xacro:property name="source" value="$(find last_letter_2)/config/param/aircrafts/plane_1wing_sensors/rigidBody.yaml" />
+<xacro:property name="source" value="$(find last_letter_2)/config/param/aircrafts/plane_1wing_sensors/mass.yaml" />
 <xacro:property name="dictionary" value="${load_yaml(source)}"/>
 <xacro:property name="mass" value="${dictionary['airframe/m']}"/>

File: last_letter_2/config/param/aircrafts/plane_3wing/urdf/model.urdf.xacro (robot description, xacro)
@@ -1,5 +1,5 @@
 <?xml version="1.0"?>
 <robot name="plane" xmlns:xacro="http://www.ros.org/wiki/xacro">
-<xacro:property name="source" value="$(find last_letter_2)/config/param/aircrafts/plane_3wing/rigidBody.yaml" />
+<xacro:property name="source" value="$(find last_letter_2)/config/param/aircrafts/plane_3wing/mass.yaml" />
 <xacro:property name="dictionary" value="${load_yaml(source)}"/>
 <xacro:property name="mass" value="${dictionary['airframe/m']}"/>

File: last_letter_2/config/param/aircrafts/quadcopter/urdf/model.urdf.xacro (robot description, xacro)
@@ -1,5 +1,5 @@
 <?xml version="1.0"?>
 <robot name="quadcopter" xmlns:xacro="http://www.ros.org/wiki/xacro">
-<xacro:property name="source" value="$(find last_letter_2)/config/param/aircrafts/quadcopter/rigidBody.yaml" />
+<xacro:property name="source" value="$(find last_letter_2)/config/param/aircrafts/quadcopter/mass.yaml" />
 <xacro:property name="dictionary" value="${load_yaml(source)}"/>
 <xacro:property name="body_mass" value="${dictionary['airframe/m']}"/>
