Commit message: Add mesh files
Add some Collada files to be uses as meshes in urdf files.

File: last_letter_2/config/param/models/plane_1wing/urdf/model.urdf.xacro (robot description, xacro)
@@ -12,7 +12,6 @@
     <link name="body_FLU">
         <visual>
-            <origin rpy="0 -${pi/2} 0 " />
-            <geometry>
-                <cylinder radius="${body_r}" length="${body_h}" />
+            <geometry>
+               <mesh filename="file:///home/me/catkin_ws/src/last_letter_2/last_letter_2/config/param/meshes/piper_pa18_dae/piper_pa18.dae"/>
             </geometry>
         </visual>
@@ -130,5 +129,5 @@
     </joint>
 <!-- propeller link parameters x, y, z, mass -->
-<xacro:property name="propeller_x" value="${0.8*body_s}" />
+<xacro:property name="propeller_x" value="${1.3*body_s}" />
 <xacro:property name="propeller_y" value="${0.2*body_s}" />
 <xacro:property name="propeller_z" value="${0.05*body_s}" />
@@ -136,6 +135,7 @@
     <link name="prop1">
         <visual>
-            <geometry>
-                <box size="${propeller_x} ${propeller_y} ${propeller_z}" />
+        <origin xyz="0 -0.149 0.01" rpy="0 0 0" />
+            <geometry>
+               <mesh filename="file:///home/me/catkin_ws/src/last_letter_2/last_letter_2/config/param/meshes/propeller.dae"/>
             </geometry>
         </visual>

File: last_letter_2/config/param/models/plane_3w_2m_electric/urdf/model.urdf.xacro (robot description, xacro)
@@ -250,6 +250,7 @@
     <link name="prop1">
         <visual>
-            <geometry>
-                <box size="${propeller_x} ${propeller_y} ${propeller_z}" />
+        <origin xyz="0 -0.149 0.01" rpy="0 0 0" />
+            <geometry>
+               <mesh filename="file:///home/me/catkin_ws/src/last_letter_2/last_letter_2/config/param/meshes/propeller.dae"/>
             </geometry>
         </visual>
@@ -273,6 +274,7 @@
     <link name="prop2">
         <visual>
-            <geometry>
-                <box size="${propeller_x} ${propeller_y} ${propeller_z}" />
+        <origin xyz="0 -0.149 0.01" rpy="0 0 0" />
+            <geometry>
+               <mesh filename="file:///home/me/catkin_ws/src/last_letter_2/last_letter_2/config/param/meshes/propeller.dae"/>
             </geometry>
         </visual>

Commit message: CSL logo in world
add the CSL logo in the simulation world

File: last_letter_2/config/param/models/plane_1wing/urdf/model.urdf.xacro (robot description, xacro)
@@ -13,5 +13,5 @@
         <visual>
             <geometry>
-               <mesh filename="file:///home/me/catkin_ws/src/last_letter_2/last_letter_2/config/param/meshes/piper_pa18_dae/piper_pa18.dae"/>
+                <cylinder radius="${body_r}" length="${body_h}" />
             </geometry>
         </visual>

Commit message: Rot diraction of motors + electricEngine
Fix some errors with rotation direction of motor and add electric engine again.

File: last_letter_2/config/param/models/plane_1wing/urdf/model.urdf.xacro (robot description, xacro)
@@ -12,4 +12,5 @@
     <link name="body_FLU">
         <visual>
+            <origin rpy="0 -${pi/2} 0 " />
             <geometry>
                 <cylinder radius="${body_r}" length="${body_h}" />

File: last_letter_2/config/param/models/quadcopter/urdf/model.urdf.xacro (robot description, xacro)
@@ -1,5 +1,5 @@
 <?xml version="1.0"?>
 <robot name="quadcopter" xmlns:xacro="http://www.ros.org/wiki/xacro">
-<xacro:property name="body_mass" value="3"/>
+<xacro:property name="body_mass" value="1.5"/>
 <!-- body, airfoil sizes -->
 <xacro:property name="body_s" value="1" />

Commit message: Small changes

File: last_letter_2/config/param/models/plane_1wing/urdf/model.urdf.xacro (robot description, xacro)
@@ -137,5 +137,5 @@
         <origin xyz="0 -0.149 0.01" rpy="0 0 0" />
             <geometry>
-               <mesh filename="file:///home/me/catkin_ws/src/last_letter_2/last_letter_2/config/param/meshes/propeller.dae"/>
+               <mesh filename="package://last_letter_2/config/param/meshes/propeller.dae"/>
             </geometry>
         </visual>

File: last_letter_2/config/param/models/plane_3wing_2motor/urdf/model.urdf.xacro (robot description, xacro)
@@ -251,5 +251,5 @@
         <origin xyz="0 -0.149 0.01" rpy="0 0 0" />
             <geometry>
-               <mesh filename="file:///home/me/catkin_ws/src/last_letter_2/last_letter_2/config/param/meshes/propeller.dae"/>
+               <mesh filename="package://last_letter_2/config/param/meshes/propeller.dae"/>
             </geometry>
         </visual>
@@ -275,5 +275,5 @@
         <origin xyz="0 -0.149 0.01" rpy="0 0 0" />
             <geometry>
-               <mesh filename="file:///home/me/catkin_ws/src/last_letter_2/last_letter_2/config/param/meshes/propeller.dae"/>
+               <mesh filename="package://last_letter_2/config/param/meshes/propeller.dae"/>
             </geometry>
         </visual>
