Commit message: Code Clean + Format

File: last_letter_2/config/param/models/hexacopter/urdf/model.urdf.xacro (robot description, xacro)
@@ -2,5 +2,5 @@
 <robot name="hexacopter" xmlns:xacro="http://www.ros.org/wiki/xacro">
 <xacro:property name="body_mass" value="3"/>
-<!-- body, airfoil sizes -->
+<!-- body, airfoil size -->
 <xacro:property name="body_s" value="1" />
 <!-- body link parameters x, y, z, mass-->
@@ -24,5 +24,5 @@
         <origin rpy="0 0 0"/>
             <mass value="${body_m}" />
-             <inertia    ixx="${1/12*body_m*body_h*body_h+1/4*body_m*body_r*body_r}" ixy="0" ixz="0" iyz="0"
+             <inertia   ixx="${1/12*body_m*body_h*body_h+1/4*body_m*body_r*body_r}" ixy="0" ixz="0" iyz="0"
                         iyy="${1/12*body_m*body_h*body_h+1/4*body_m*body_r*body_r}"
                         izz="${1/2*body_m*body_r*body_r}" />
@@ -112,5 +112,5 @@
         <child link="arm3" />
     </joint>
-        <link name="arm4">
+    <link name="arm4">
         <visual>
         <origin xyz="${arm_x/2} 0 0"/>
@@ -138,5 +138,5 @@
         <child link="arm4" />
     </joint>
-     <link name="arm5">
+    <link name="arm5">
         <visual>
         <origin xyz="${arm_x/2} 0 0"/>
@@ -164,5 +164,5 @@
         <child link="arm5" />
     </joint>
-     <link name="arm6">
+    <link name="arm6">
         <visual>
         <origin xyz="${arm_x/2} 0 0"/>
@@ -195,5 +195,5 @@
 <xacro:property name="motor_m" value="${0.1*body_m}" />
 <!-- only motor(Number_0f_Motor) acceptable name for motors -->
-     <link name="motor1">
+    <link name="motor1">
         <visual>
         <origin xyz="${motor_r/2} 0 0" rpy="0 ${pi/2} 0"/>
@@ -220,7 +220,7 @@
         <parent link="arm1" />
         <child link="motor1" />
-        <limit effort="1000.0" velocity="0.5"/>
-    </joint>
-     <link name="motor2">
+        <limit effort="1000.0" velocity="0.5"/>  --default limits upper=lower=0
+    </joint>
+    <link name="motor2">
         <visual>
         <origin xyz="${motor_r/2} 0 0" rpy="0 ${pi/2} 0"/>
@@ -247,7 +247,7 @@
         <parent link="arm2" />
         <child link="motor2" />
-        <limit effort="1000.0" velocity="0.5"/>
-    </joint>
-     <link name="motor3">
+        <limit effort="1000.0" velocity="0.5"/>  --default limits upper=lower=0
+    </joint>
+    <link name="motor3">
         <visual>
         <origin xyz="${motor_r/2} 0 0" rpy="0 ${pi/2} 0"/>
@@ -274,7 +274,7 @@
         <parent link="arm3" />
         <child link="motor3" />
-        <limit effort="1000.0" velocity="0.5"/>
-    </joint>
-     <link name="motor4">
+        <limit effort="1000.0" velocity="0.5"/>  --default limits upper=lower=0
+    </joint>
+    <link name="motor4">
         <visual>
         <origin xyz="${motor_r/2} 0 0" rpy="0 ${pi/2} 0"/>
@@ -301,5 +301,5 @@
         <parent link="arm4" />
         <child link="motor4" />
-        <limit effort="1000.0" velocity="0.5"/>
+        <limit effort="1000.0" velocity="0.5"/>  --default limits upper=lower=0
     </joint>
          <link name="motor5">
@@ -328,7 +328,7 @@
         <parent link="arm5" />
         <child link="motor5" />
-        <limit effort="1000.0" velocity="0.5"/>
-    </joint>
-         <link name="motor6">
+        <limit effort="1000.0" velocity="0.5"/>  --default limits upper=lower=0
+    </joint>
+    <link name="motor6">
         <visual>
         <origin xyz="${motor_r/2} 0 0" rpy="0 ${pi/2} 0"/>
@@ -355,5 +355,5 @@
         <parent link="arm6" />
         <child link="motor6" />
-        <limit effort="1000.0" velocity="0.5"/>
+        <limit effort="1000.0" velocity="0.5"/>  --default limits upper=lower=0
     </joint>
  -------------------------------------------------------------- axles
@@ -530,5 +530,5 @@
 <xacro:property name="propeller_y" value="${body_s/10}" />
 <xacro:property name="propeller_z" value="${body_s/40}" />
-   <link name="prop1">
+    <link name="prop1">
         <visual>
             <origin xyz="0 0 0" rpy="0 ${pi/2} 0"/>
@@ -557,5 +557,5 @@
         <child link="prop1" />
     </joint>
-   <link name="prop2">
+    <link name="prop2">
         <visual>
             <origin xyz="0 0 0" rpy="0 ${pi/2} 0"/>
@@ -584,5 +584,5 @@
         <child link="prop2" />
     </joint>
-   <link name="prop3">
+    <link name="prop3">
         <visual>
             <origin xyz="0 0 0" rpy="0 ${pi/2} 0"/>
@@ -611,5 +611,5 @@
         <child link="prop3" />
     </joint>
-   <link name="prop4">
+    <link name="prop4">
         <visual>
             <origin xyz="0 0 0" rpy="0 ${pi/2} 0"/>
@@ -638,5 +638,5 @@
         <child link="prop4" />
     </joint>
-   <link name="prop5">
+    <link name="prop5">
         <visual>
             <origin xyz="0 0 0" rpy="0 ${pi/2} 0"/>
@@ -665,5 +665,5 @@
         <child link="prop5" />
     </joint>
-   <link name="prop6">
+    <link name="prop6">
         <visual>
             <origin xyz="0 0 0" rpy="0 ${pi/2} 0"/>
@@ -692,12 +692,12 @@
         <child link="prop6" />
     </joint>
-    --------------------------------------------------------------model plugins
+    <!-- model plugins -->
     <gazebo>
-    <plugin name="model_plugin" filename="libmodel_plugin.so"/>
-    <plugin name="joint_state_publisher" filename="libgazebo_ros_joint_state_publisher.so">
-        <jointName>arm1_to_motor1, arm2_to_motor2, arm3_to_motor3,arm4_to_motor4,arm5_to_motor5,arm6_to_motor6,motor1_to_axle1,motor2_to_axle2,motor3_to_axle3,motor4_to_axle4,motor5_to_axle5,motor6_to_axle6 </jointName>
-        <robotNamespace>last_letter_2</robotNamespace>
-        <updateRate>0</updateRate>
-    </plugin>
-  </gazebo>
+        <plugin name="model_plugin" filename="libmodel_plugin.so"/>
+        <plugin name="joint_state_publisher" filename="libgazebo_ros_joint_state_publisher.so">
+            <jointName>arm1_to_motor1, arm2_to_motor2, arm3_to_motor3,arm4_to_motor4,arm5_to_motor5,arm6_to_motor6,motor1_to_axle1,motor2_to_axle2,motor3_to_axle3,motor4_to_axle4,motor5_to_axle5,motor6_to_axle6 </jointName>
+            <robotNamespace>last_letter_2</robotNamespace>
+            <updateRate>0</updateRate>
+        </plugin>
+    </gazebo>
 </robot>

File: last_letter_2/config/param/models/plane_1wing/urdf/model.urdf.xacro (robot description, xacro)
@@ -1,8 +1,7 @@
 <?xml version="1.0"?>
-<robot name="plane" xmlns:xacro="http://www.ros.org/wiki/xacro">
+<robot name="plane_1wing" xmlns:xacro="http://www.ros.org/wiki/xacro">
 <xacro:property name="mass" value="3"/>
-<!-- body, airfoil sizes -->
+<!-- body, airfoil size -->
 <xacro:property name="body_s" value="1" />
-<xacro:property name="airfoil_s" value="1" />
 <!-- body link , body_height, body_rad, body_mass -->
 <xacro:property name="body_h" value="${2.5*body_s}" />
@@ -33,8 +32,8 @@
     ----------------------------------------------------------------------------  airfoils
 <!-- airfoil1 link parameters , x, y, z, mass-->
-<xacro:property name="airfoil_x" value="${airfoil_s/2}" />
-<xacro:property name="airfoil_y" value="${airfoil_s*6}" />
-<xacro:property name="airfoil_z" value="${airfoil_s/10}"/>
-<xacro:property name="airfoil_m" value="${0.3*mass}" />               ----airfoil mass
+<xacro:property name="airfoil_x" value="${body_s/2}" />
+<xacro:property name="airfoil_y" value="${body_s*6}" />
+<xacro:property name="airfoil_z" value="${body_s/10}"/>
+<xacro:property name="airfoil_m" value="${0.3*mass}" />
     <!-- only airfoil(Number_0f_Airfoil) acceptable name for airfoils -->
     <link name="airfoil1">
@@ -70,5 +69,5 @@
 <xacro:property name="motor_m" value="${0.3*mass}" />
 <!-- only motor(Number_0f_Motor) acceptable name for motors -->
- <link name="motor1">
+    <link name="motor1">
         <visual>
             <origin xyz="${0.5*motor_x} 0 0"/>
@@ -93,5 +92,5 @@
     <joint name="body_FLU_to_motor1" type="revolute">
         <origin xyz="${0.5*body_h} 0 0" rpy="0 0 0" />
-        <limit effort="1000.0" velocity="0.5"/>
+        <limit effort="1000.0" velocity="0.5"/>  --default limits upper=lower=0
         <parent link="body_FLU" />
         <child link="motor1" />
@@ -277,12 +276,12 @@
         <child link="rear_wheel" />
     </joint>
-<!-- model plugins -->
+    <!-- model plugins -->
     <gazebo>
-    <plugin name="model_plugin" filename="libmodel_plugin.so"/>
-    <plugin name="joint_state_publisher" filename="libgazebo_ros_joint_state_publisher.so">
-        <jointName>body_FLU_to_airfoil1, body_FLU_to_motor1, motor1_to_axle1, wheel_base_to_left_wheel, wheel_base_to_right_wheel, body_FLU_to_rear_wheel </jointName>
-        <robotNamespace>last_letter_2</robotNamespace>
-        <updateRate>0</updateRate>
-    </plugin>
-  </gazebo>
+        <plugin name="model_plugin" filename="libmodel_plugin.so"/>
+        <plugin name="joint_state_publisher" filename="libgazebo_ros_joint_state_publisher.so">
+            <jointName>body_FLU_to_airfoil1, body_FLU_to_motor1, motor1_to_axle1, wheel_base_to_left_wheel, wheel_base_to_right_wheel, body_FLU_to_rear_wheel </jointName>
+            <robotNamespace>last_letter_2</robotNamespace>
+            <updateRate>0</updateRate>
+        </plugin>
+    </gazebo>
 </robot>
