Commit message: Code Clean + Format

File: last_letter_2/config/param/models/plane_1wing_sensors/urdf/model.urdf.xacro (robot description, xacro)
@@ -1,66 +1,66 @@
 <?xml version="1.0"?>
-<robot name="plane_sensors" xmlns:xacro="http://www.ros.org/wiki/xacro">
+<robot name="plane_1wing_sensors" xmlns:xacro="http://www.ros.org/wiki/xacro">
+<!-- total model mass -->
 <xacro:property name="mass" value="3"/>
 <!-- body, airfoil sizes -->
 <xacro:property name="body_s" value="1" />
-<xacro:property name="airfoil_s" value="1" />
 <!-- body link , body_height, body_rad, body_mass -->
 <xacro:property name="body_h" value="${2.5*body_s}" />
 <xacro:property name="body_r" value="${0.5*body_s}" />
 <xacro:property name="body_m" value="${0.3*mass}" />
-    <!-- only body_FLU acceptable name for base_link -->
-    <link name="body_FLU">
-        <visual>
-            <origin rpy="0 -${pi/2} 0 " />
-            <geometry>
-                <cylinder radius="${body_r}" length="${body_h}" />
-            </geometry>
-        </visual>
-        <collision>
-            <origin rpy="0 -${pi/2} 0 " />
-            <geometry>
-                <cylinder radius="${body_r}" length="${body_h}" />
-            </geometry>
-        </collision>
-        <inertial>
-            <origin rpy="0 -${pi/2} 0 " />
-            <mass value="${body_m}" />
-            <inertia    ixx="${1/12*(3*body_r*body_r+body_h*body_h)*body_m}" ixy="0" ixz="0" iyz="0"
-                        iyy="${1/12*(3*body_r*body_r+body_h*body_h)*body_m}"
-                        izz="${1/2*body_m*body_r*body_r}" />
-        </inertial>
-    </link>
+  <!-- only body_FLU acceptable name for base_link -->
+  <link name="body_FLU">
+    <visual>
+      <origin rpy="0 -${pi/2} 0 " />
+      <geometry>
+        <cylinder radius="${body_r}" length="${body_h}" />
+      </geometry>
+    </visual>
+    <collision>
+      <origin rpy="0 -${pi/2} 0 " />
+      <geometry>
+        <cylinder radius="${body_r}" length="${body_h}" />
+      </geometry>
+    </collision>
+    <inertial>
+      <origin rpy="0 -${pi/2} 0 " />
+      <mass value="${body_m}" />
+      <inertia  ixx="${1/12*(3*body_r*body_r+body_h*body_h)*body_m}" ixy="0" ixz="0" iyz="0"
+                iyy="${1/12*(3*body_r*body_r+body_h*body_h)*body_m}"
+                izz="${1/2*body_m*body_r*body_r}" />
+    </inertial>
+  </link>
     ----------------------------------------------------------------------------  airfoils
 <!-- airfoil1 link parameters , x, y, z, mass-->
-<xacro:property name="airfoil_x" value="${airfoil_s/2}" />
-<xacro:property name="airfoil_y" value="${airfoil_s*6}" />
-<xacro:property name="airfoil_z" value="${airfoil_s/10}"/>
+<xacro:property name="airfoil_x" value="${body_s/2}" />
+<xacro:property name="airfoil_y" value="${body_s*6}" />
+<xacro:property name="airfoil_z" value="${body_s/10}"/>
 <xacro:property name="airfoil_m" value="${0.3*mass}" />               ----airfoil mass
-    <!-- only airfoil(Number_0f_Airfoil) acceptable name for airfoils -->
-    <link name="airfoil1">
-        <visual>
-            <geometry>
-                <box size="${airfoil_x} ${airfoil_y} ${airfoil_z}" />
-            </geometry>
-        </visual>
-        <collision>
-            <geometry>
-                <box size="${airfoil_x} ${airfoil_y} ${airfoil_z}" />
-            </geometry>
-        </collision>
-         <inertial>
-            <mass value="${airfoil_m}" />
-            <inertia    ixx="${1/12*airfoil_m*(airfoil_y*airfoil_y+airfoil_z*airfoil_z)}" ixy="0" ixz="0" iyz="0"
-                        iyy="${1/12*airfoil_m*(airfoil_x*airfoil_x+airfoil_z*airfoil_z)}"
-                        izz="${1/12*airfoil_m*(airfoil_x*airfoil_x+airfoil_y*airfoil_y)}" />
-        </inertial>
-    </link>
-    <joint name="body_FLU_to_airfoil1" type="revolute">
-        <origin xyz="0 0 0" rpy ="0 0 0"/>
-        <parent link="body_FLU" />
-        <child link="airfoil1" />
-        <limit effort="1000.0" velocity="0.5"/>   ---default limits upper=lower=0
-    </joint>
-    ----------------------------------------------------------------------------------- motors
+  <!-- only airfoil(Number_0f_Airfoil) acceptable name for airfoils -->
+  <link name="airfoil1">
+    <visual>
+      <geometry>
+        <box size="${airfoil_x} ${airfoil_y} ${airfoil_z}" />
+      </geometry>
+    </visual>
+    <collision>
+      <geometry>
+      <box size="${airfoil_x} ${airfoil_y} ${airfoil_z}" />
+      </geometry>
+    </collision>
+    <inertial>
+      <mass value="${airfoil_m}" />
+      <inertia  ixx="${1/12*airfoil_m*(airfoil_y*airfoil_y+airfoil_z*airfoil_z)}" ixy="0" ixz="0" iyz="0"
+                iyy="${1/12*airfoil_m*(airfoil_x*airfoil_x+airfoil_z*airfoil_z)}"
+                izz="${1/12*airfoil_m*(airfoil_x*airfoil_x+airfoil_y*airfoil_y)}" />
+    </inertial>
+  </link>
+  <joint name="body_FLU_to_airfoil1" type="revolute">
+    <origin xyz="0 0 0" rpy ="0 0 0"/>
+    <parent link="body_FLU" />
+    <child link="airfoil1" />
+    <limit effort="1000.0" velocity="0.5"/> ---default limits upper=lower=0
+  </joint>
+  ----------------------------------------------------------------------------------- motors
 <!-- motor link -->
 <!-- motor parameters , x, y, z, mass -->
@@ -70,63 +70,63 @@
 <xacro:property name="motor_m" value="${0.3*mass}" />
 <!-- only motor(Number_0f_Motor) acceptable name for motors -->
- <link name="motor1">
-        <visual>
-            <origin xyz="${0.5*motor_x} 0 0"/>
-            <geometry>
-                <box size="${motor_x} ${motor_y} ${motor_z}" />
-            </geometry>
-        </visual>
-        <collision>
-            <origin xyz="${0.5*motor_x} 0 0"/>
-            <geometry>
-                <box size="${motor_x} ${motor_y} ${motor_z}" />
-            </geometry>
-        </collision>
-        <inertial>
-            <origin xyz="${0.5*motor_x} 0 0"/>
-            <mass value="${motor_m}" />
-            <inertia    ixx="${1/12*motor_m*(motor_y*motor_y+motor_z*motor_z)}" ixy="0" ixz="0" iyz="0"
-                        iyy="${1/12*motor_m*(motor_x*motor_x+motor_z*motor_z)}"
-                        izz="${1/12*motor_m*(motor_x*motor_x+motor_y*motor_y)}" />
-        </inertial>
-    </link>
-    <joint name="body_FLU_to_motor1" type="revolute">
-        <origin xyz="${0.5*body_h} 0 0" rpy="0 0 0" />
-        <limit effort="1000.0" velocity="0.5"/>
-        <parent link="body_FLU" />
-        <child link="motor1" />
-    </joint>
- -----------------------------------------------------------------------------------propeller
+  <link name="motor1">
+    <visual>
+      <origin xyz="${0.5*motor_x} 0 0"/>
+      <geometry>
+        <box size="${motor_x} ${motor_y} ${motor_z}" />
+      </geometry>
+    </visual>
+    <collision>
+      <origin xyz="${0.5*motor_x} 0 0"/>
+      <geometry>
+        <box size="${motor_x} ${motor_y} ${motor_z}" />
+      </geometry>
+    </collision>
+    <inertial>
+      <origin xyz="${0.5*motor_x} 0 0"/>
+      <mass value="${motor_m}" />
+      <inertia  ixx="${1/12*motor_m*(motor_y*motor_y+motor_z*motor_z)}" ixy="0" ixz="0" iyz="0"
+                iyy="${1/12*motor_m*(motor_x*motor_x+motor_z*motor_z)}"
+                izz="${1/12*motor_m*(motor_x*motor_x+motor_y*motor_y)}" />
+    </inertial>
+  </link>
+  <joint name="body_FLU_to_motor1" type="revolute">
+    <origin xyz="${0.5*body_h} 0 0" rpy="0 0 0" />
+    <limit effort="1000.0" velocity="0.5"/>  --default limits upper=lower=0
+    <parent link="body_FLU" />
+    <child link="motor1" />
+  </joint>
+-----------------------------------------------------------------------------------propeller
 <!-- axle link parameters height, rad, mass-->
 <xacro:property name="axle_h" value="${body_h/12}" />
 <xacro:property name="axle_r" value="${body_r/10}" />
 <xacro:property name="axle_m" value="${0.005*mass}" />
-    <link name="axle1">
-        <visual>
-            <origin xyz="${axle_h/2} 0 0" rpy="0 ${pi/2} 0"/>
-            <geometry>
-                <cylinder radius="${axle_r}" length="${axle_h}" />
-            </geometry>
-        </visual>
-        <collision>
-            <origin xyz="${axle_h/2} 0 0" rpy="0 ${pi/2} 0"/>
-            <geometry>
-                <cylinder radius="${axle_r}" length="${axle_h}" />
-            </geometry>
-        </collision>
-        <inertial>
-            <origin xyz="${axle_h/2} 0 0" />
-            <mass value="${axle_m}" />
-            <inertia    ixx="${1/12*axle_m*axle_h*axle_h+1/4*axle_m*axle_r*axle_r}" ixy="0" ixz="0" iyz="0"
-                        iyy="${1/12*axle_m*axle_h*axle_h+1/4*axle_m*axle_r*axle_r}"
-                        izz="${1/2*axle_m*axle_r*axle_r}" />
-        </inertial>
-    </link>
-    <joint name="motor1_to_axle1" type="continuous">
-        <origin xyz="${motor_x} 0 0" rpy="0 0 0" />
-        <axis xyz="1 0 0" />
-        <parent link="motor1" />
-        <child link="axle1" />
-    </joint>
+  <link name="axle1">
+    <visual>
+      <origin xyz="${axle_h/2} 0 0" rpy="0 ${pi/2} 0"/>
+      <geometry>
+        <cylinder radius="${axle_r}" length="${axle_h}" />
+      </geometry>
+    </visual>
+    <collision>
+      <origin xyz="${axle_h/2} 0 0" rpy="0 ${pi/2} 0"/>
+      <geometry>
+        <cylinder radius="${axle_r}" length="${axle_h}" />
+      </geometry>
+    </collision>
+    <inertial>
+      <origin xyz="${axle_h/2} 0 0" />
+      <mass value="${axle_m}" />
+      <inertia  ixx="${1/12*axle_m*axle_h*axle_h+1/4*axle_m*axle_r*axle_r}" ixy="0" ixz="0" iyz="0"
+                iyy="${1/12*axle_m*axle_h*axle_h+1/4*axle_m*axle_r*axle_r}"
+                izz="${1/2*axle_m*axle_r*axle_r}" />
+    </inertial>
+  </link>
+  <joint name="motor1_to_axle1" type="continuous">
+    <origin xyz="${motor_x} 0 0" rpy="0 0 0" />
+    <axis xyz="1 0 0" />
+    <parent link="motor1" />
+    <child link="axle1" />
+  </joint>
 <!-- propeller link parameters x, y, z, mass -->
 <xacro:property name="propeller_x" value="${0.8*body_s}" />
@@ -134,147 +134,147 @@
 <xacro:property name="propeller_z" value="${0.05*body_s}" />
 <xacro:property name="propeller_m" value="${0.015*mass}" />
-    <link name="prop1">
-        <visual>
-            <geometry>
-                <box size="${propeller_x} ${propeller_y} ${propeller_z}" />
-            </geometry>
-        </visual>
-        <collision>
-            <geometry>
-                <box size="${propeller_x} ${propeller_y} ${propeller_z}" />
-            </geometry>
-        </collision>
-        <inertial>
-            <mass value="${propeller_m}" />
-           <inertia     ixx="${1/12*propeller_m*(propeller_y*propeller_y+propeller_z*propeller_z)}" ixy="0" ixz="0" iyz="0"
-                        iyy="${1/12*propeller_m*(propeller_x*propeller_x+propeller_z*propeller_z)}"
-                        izz="${1/12*propeller_m*(propeller_x*propeller_x+propeller_y*propeller_y)}" />
-        </inertial>
-    </link>
-    <joint name="axle1_to_propeller1" type="fixed">
-        <origin xyz="${axle_h} 0 0" rpy="0 ${pi/2} 0" />
-        <parent link="axle1" />
-        <child link="prop1" />
-    </joint>
-     ---------------------------------------------------------------------------front wheels
-     <!-- wheel_base_link parameters, x, y, z, mass-->
+  <link name="prop1">
+    <visual>
+      <geometry>
+        <box size="${propeller_x} ${propeller_y} ${propeller_z}" />
+      </geometry>
+    </visual>
+    <collision>
+      <geometry>
+        <box size="${propeller_x} ${propeller_y} ${propeller_z}" />
+      </geometry>
+    </collision>
+    <inertial>
+      <mass value="${propeller_m}" />
+      <inertia  ixx="${1/12*propeller_m*(propeller_y*propeller_y+propeller_z*propeller_z)}" ixy="0" ixz="0" iyz="0"
+                iyy="${1/12*propeller_m*(propeller_x*propeller_x+propeller_z*propeller_z)}"
+                izz="${1/12*propeller_m*(propeller_x*propeller_x+propeller_y*propeller_y)}" />
+    </inertial>
+  </link>
+  <joint name="axle1_to_propeller1" type="fixed">
+    <origin xyz="${axle_h} 0 0" rpy="0 ${pi/2} 0" />
+    <parent link="axle1" />
+    <child link="prop1" />
+  </joint>
+    ---------------------------------------------------------------------------front wheels
+    <!-- wheel_base_link parameters, x, y, z, mass-->
 <xacro:property name="wheel_base_x" value="${0.05*body_s}" />
 <xacro:property name="wheel_base_y" value="${2*body_s}" />
 <xacro:property name="wheel_base_z" value="${0.05*body_s}" />
 <xacro:property name="wheel_base_m" value="${0.05*mass}" />
-    <link name="wheel_base">
-        <visual>
-            <geometry>
-                <box size="${wheel_base_x} ${wheel_base_y} ${wheel_base_z}" />
-            </geometry>
-        </visual>
-        <collision>
-            <geometry>
-                <box size="${wheel_base_x} ${wheel_base_y} ${wheel_base_z}" />
-            </geometry>
-        </collision>
-        <inertial>
-            <mass value="${wheel_base_m}" />
-            <inertia    ixx="${1/12*wheel_base_m*(wheel_base_y*wheel_base_y+wheel_base_z*wheel_base_z)}" ixy="0" ixz="0" iyz="0"
-                        iyy="${1/12*wheel_base_m*(wheel_base_x*wheel_base_x+wheel_base_z*wheel_base_z)}"
-                        izz="${1/12*wheel_base_m*(wheel_base_x*wheel_base_x+wheel_base_y*propeller_y)}" />
-        </inertial>
-    </link>
-    <joint name=" body_FLU_to_wheel_base" type="fixed">
-        <origin xyz="${0.4*body_h} 0 -${body_r}" rpy="0 0 0" />
-        <parent link="body_FLU" />
-        <child link="wheel_base" />
-    </joint>
+  <link name="wheel_base">
+    <visual>
+      <geometry>
+        <box size="${wheel_base_x} ${wheel_base_y} ${wheel_base_z}" />
+      </geometry>
+    </visual>
+    <collision>
+      <geometry>
+        <box size="${wheel_base_x} ${wheel_base_y} ${wheel_base_z}" />
+      </geometry>
+    </collision>
+    <inertial>
+      <mass value="${wheel_base_m}" />
+      <inertia  ixx="${1/12*wheel_base_m*(wheel_base_y*wheel_base_y+wheel_base_z*wheel_base_z)}" ixy="0" ixz="0" iyz="0"
+                iyy="${1/12*wheel_base_m*(wheel_base_x*wheel_base_x+wheel_base_z*wheel_base_z)}"
+                izz="${1/12*wheel_base_m*(wheel_base_x*wheel_base_x+wheel_base_y*propeller_y)}" />
+    </inertial>
+  </link>
+  <joint name=" body_FLU_to_wheel_base" type="fixed">
+    <origin xyz="${0.4*body_h} 0 -${body_r}" rpy="0 0 0" />
+    <parent link="body_FLU" />
+    <child link="wheel_base" />
+  </joint>
 <!-- left wheel link parameters, rad, height, mass-->
 <xacro:property name="left_wheel_r" value="${0.3*body_s}" />
 <xacro:property name="left_wheel_h" value="${0.1*body_s}" />
 <xacro:property name="left_wheel_m" value="${0.01*mass}" />
-    <link name="left_wheel">
-        <visual>
-            <origin xyz="0 0 ${left_wheel_h/2}" />
-            <geometry>
-                <cylinder radius="${left_wheel_r}" length="${left_wheel_h}" />
-            </geometry>
-        </visual>
-        <collision>
-            <origin xyz="0 0 ${left_wheel_h/2}" />
-            <geometry>
-                <cylinder radius="${left_wheel_r}" length="${left_wheel_h}" />
-            </geometry>
-        </collision>
-        <inertial>
-            <origin xyz="0 0 ${left_wheel_h/2}" />
-            <mass value="${left_wheel_m}" />
-           <inertia     ixx="${1/12*left_wheel_m*left_wheel_h*left_wheel_h+1/4*left_wheel_m*left_wheel_r*left_wheel_r}" ixy="0" ixz="0" iyz="0"
-                        iyy="${1/12*left_wheel_m*left_wheel_h*left_wheel_h+1/4*left_wheel_m*left_wheel_r*left_wheel_r}"
-                        izz="${1/2*left_wheel_m*left_wheel_r*left_wheel_r}" />
-        </inertial>
-    </link>
-    <joint name="wheel_base_to_left_wheel" type="continuous">
-        <origin xyz="0 -${wheel_base_y/2} 0" rpy="${pi/2} 0 0" />
-        <parent link="wheel_base" />
-        <child link="left_wheel" />
-        <axis xyz=" 0 0 1" />
-    </joint>
+  <link name="left_wheel">
+    <visual>
+      <origin xyz="0 0 ${left_wheel_h/2}" />
+      <geometry>
+        <cylinder radius="${left_wheel_r}" length="${left_wheel_h}" />
+      </geometry>
+    </visual>
+    <collision>
+      <origin xyz="0 0 ${left_wheel_h/2}" />
+      <geometry>
+        <cylinder radius="${left_wheel_r}" length="${left_wheel_h}" />
+      </geometry>
+    </collision>
+    <inertial>
+      <origin xyz="0 0 ${left_wheel_h/2}" />
+      <mass value="${left_wheel_m}" />
+      <inertia  ixx="${1/12*left_wheel_m*left_wheel_h*left_wheel_h+1/4*left_wheel_m*left_wheel_r*left_wheel_r}" ixy="0" ixz="0" iyz="0"
+                iyy="${1/12*left_wheel_m*left_wheel_h*left_wheel_h+1/4*left_wheel_m*left_wheel_r*left_wheel_r}"
+                izz="${1/2*left_wheel_m*left_wheel_r*left_wheel_r}" />
+    </inertial>
+  </link>
+  <joint name="wheel_base_to_left_wheel" type="continuous">
+    <origin xyz="0 -${wheel_base_y/2} 0" rpy="${pi/2} 0 0" />
+    <parent link="wheel_base" />
+    <child link="left_wheel" />
+    <axis xyz=" 0 0 1" />
+  </joint>
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
File: last_letter_2/config/param/models/plane_3wing_2motor/urdf/model.urdf.xacro (robot description, xacro)
@@ -1,8 +1,7 @@
 <?xml version="1.0"?>
-<robot name="plane" xmlns:xacro="http://www.ros.org/wiki/xacro">
+<robot name="plane_3wing_2motor" xmlns:xacro="http://www.ros.org/wiki/xacro">
 <xacro:property name="mass" value="3"/>
 <!-- body, airfoil sizes -->
 <xacro:property name="body_s" value="1" />
-<xacro:property name="airfoil_s" value="1" />
 <!-- body link , body_height, body_rad, body_mass -->
 <xacro:property name="body_h" value="${2.5*body_s}" />
@@ -32,9 +31,9 @@
     </link>
     ----------------------------------------------------------------------------  airfoils
-<!-- airfoil1 link parameters , x, y, z, mass-->
-<xacro:property name="airfoil_x" value="${airfoil_s/2}" />
-<xacro:property name="airfoil_y" value="${airfoil_s*6}" />
-<xacro:property name="airfoil_z" value="${airfoil_s/10}"/>
-<xacro:property name="airfoil_m" value="${0.3*mass}" />               ----airfoil mass
+<!-- airfoil1 link parameters x, y, z, mass-->
+<xacro:property name="airfoil_x" value="${body_s/2}" />
+<xacro:property name="airfoil_y" value="${body_s*6}" />
+<xacro:property name="airfoil_z" value="${body_s/10}"/>
+<xacro:property name="airfoil_m" value="${0.3*mass}" />
     <!-- only airfoil(Number_0f_Airfoil) acceptable name for airfoils -->
     <link name="airfoil1">
@@ -62,5 +61,5 @@
         <limit effort="1000.0" velocity="0.5"/>   ---default limits upper=lower=0
     </joint>
- <!-- airfoil2 link parameters , x, y, z, mass-->
+ <!-- airfoil2 link parameters x, y, z, mass-->
 <xacro:property name="airfoil2_x" value="${0.3*body_s}" />
 <xacro:property name="airfoil2_y" value="${2*body_s}" />
@@ -92,5 +91,5 @@
         <limit effort="1000.0" velocity="0.5"/>   ---default limits upper=lower=0
     </joint>
-<!-- airfoil3 link parameters , x, y, z, mass-->
+<!-- airfoil3 link parameters x, y, z, mass-->
 <xacro:property name="airfoil3_x" value="${0.3*body_s}" />
 <xacro:property name="airfoil3_y" value="${0.5*body_s}" />
@@ -124,5 +123,5 @@
 ----------------------------------------------------------------------------------- motors
 <!-- motor link -->
-<!-- motor parameters , x, y, z, mass -->
+<!-- motor parameters x, y, z, mass -->
 <xacro:property name="motor_x" value="${body_s/10}" />
 <xacro:property name="motor_y" value="${body_s/5}" />
@@ -130,5 +129,5 @@
 <xacro:property name="motor_m" value="${0.3*mass}" />
 <!-- only motor(Number_0f_Motor) acceptable name for motors -->
- <link name="motor1">
+    <link name="motor1">
         <visual>
             <origin xyz="${0.5*motor_x} 0 0"/>
@@ -153,9 +152,9 @@
     <joint name="airfoil1_to_motor1" type="revolute">
         <origin xyz="${airfoil_x/2} ${0.3*airfoil_y} 0" rpy="0 0 0" />
-        <limit effort="1000.0" velocity="0.5"/>
+        <limit effort="1000.0" velocity="0.5"/>  --default limits upper=lower=0
         <parent link="airfoil1" />
         <child link="motor1" />
     </joint>
-     <link name="motor2">
+    <link name="motor2">
         <visual>
             <origin xyz="${0.5*motor_x} 0 0"/>
@@ -180,5 +179,5 @@
     <joint name="airfoil1_to_motor2" type="revolute">
         <origin xyz="${airfoil_x/2} -${0.3*airfoil_y} 0" rpy="0 0 0" />
-        <limit effort="1000.0" velocity="0.5"/>
+        <limit effort="1000.0" velocity="0.5"/>  --default limits upper=lower=0
         <parent link="airfoil1" />
         <child link="motor2" />
@@ -216,5 +215,5 @@
         <child link="axle1" />
     </joint>
-     <link name="axle2">
+    <link name="axle2">
         <visual>
             <origin xyz="${axle_h/2} 0 0" rpy="0 ${pi/2} 0"/>
@@ -417,10 +416,10 @@
 <!-- model plugins -->
     <gazebo>
-    <plugin name="model_plugin" filename="libmodel_plugin.so"/>
-    <plugin name="joint_state_publisher" filename="libgazebo_ros_joint_state_publisher.so">
-        <jointName>body_FLU_to_airfoil1,body_FLU_to_airfoil2,body_FLU_to_airfoil3, airfoil1_to_motor1, airfoil1_to_motor2, motor1_to_axle1, motor2_to_axle2, wheel_base_to_left_wheel, wheel_base_to_right_wheel, body_FLU_to_rear_wheel </jointName>
-        <robotNamespace>last_letter_2</robotNamespace>
-        <updateRate>0</updateRate>
-    </plugin>
-  </gazebo>
+        <plugin name="model_plugin" filename="libmodel_plugin.so"/>
+        <plugin name="joint_state_publisher" filename="libgazebo_ros_joint_state_publisher.so">
+            <jointName>body_FLU_to_airfoil1,body_FLU_to_airfoil2,body_FLU_to_airfoil3, airfoil1_to_motor1, airfoil1_to_motor2, motor1_to_axle1, motor2_to_axle2, wheel_base_to_left_wheel, wheel_base_to_right_wheel, body_FLU_to_rear_wheel </jointName>
+            <robotNamespace>last_letter_2</robotNamespace>
+            <updateRate>0</updateRate>
+        </plugin>
+    </gazebo>
 </robot>
