Commit message: copter controllers
Fix some details in multirotor's controller algorithm.

File: last_letter_2/config/param/models/hexacopter/urdf/model.urdf.xacro (robot description, xacro)
@@ -5,7 +5,7 @@
 <xacro:property name="body_s" value="1" />
 <!-- body link parameters x, y, z, mass-->
-<xacro:property name="body_r" value="${body_s/2}" />
-<xacro:property name="body_h" value="${body_s/8}" />
-<xacro:property name="body_m" value="${body_mass}" />
+<xacro:property name="body_r" value="${0.05*body_s}" />
+<xacro:property name="body_h" value="${0.03*body_s}" />
+<xacro:property name="body_m" value="${0.5*body_mass}" />
     <link name="body_FLU">
         <visual>
@@ -30,8 +30,8 @@
     </link>
 ---------------------------------------------------------- 6 quadcopter arms
-<xacro:property name="arm_x" value="${2*body_s}" />
-<xacro:property name="arm_y" value="${0.1*body_s}" />
-<xacro:property name="arm_z" value="${0.1*body_s}" />
-<xacro:property name="arm_m" value="${0.1*body_m}" />
+<xacro:property name="arm_x" value="${0.3*body_s}" />
+<xacro:property name="arm_y" value="${0.01*body_s}" />
+<xacro:property name="arm_z" value="${0.02*body_s}" />
+<xacro:property name="arm_m" value="${0.05*body_m}" />
     <link name="arm1">
         <visual>
@@ -191,23 +191,23 @@
     </joint>
     -------------------------------------------------------------------------- motors
-<xacro:property name="motor_r" value="${body_s/10}" />
-<xacro:property name="motor_h" value="${body_s/10}" />
-<xacro:property name="motor_m" value="${0.1*body_m}" />
+<xacro:property name="motor_r" value="${0.01*body_s}" />
+<xacro:property name="motor_h" value="${0.005*body_s}" />
+<xacro:property name="motor_m" value="${0.03*body_m}" />
 <!-- only motor(Number_0f_Motor) acceptable name for motors -->
     <link name="motor1">
         <visual>
-        <origin xyz="${motor_r/2} 0 0" rpy="0 ${pi/2} 0"/>
-            <geometry>
-                <cylinder radius="${motor_r}" length="${motor_h}" />
-            </geometry>
-        </visual>
-        <collision>
-            <origin xyz="${motor_r/2} 0 0" rpy="0 ${pi/2} 0"/>
-            <geometry>
-                <cylinder radius="${motor_r}" length="${motor_h}" />
-            </geometry>
-        </collision>
-        <inertial>
-            <origin xyz="${motor_r/2} 0 0" rpy="0 ${pi/2} 0"/>
+        <origin xyz="${motor_h/2} 0 0" rpy="0 ${pi/2} 0"/>
+            <geometry>
+                <cylinder radius="${motor_r}" length="${motor_h}" />
+            </geometry>
+        </visual>
+        <collision>
+            <origin xyz="${motor_h/2} 0 0" rpy="0 ${pi/2} 0"/>
+            <geometry>
+                <cylinder radius="${motor_r}" length="${motor_h}" />
+            </geometry>
+        </collision>
+        <inertial>
+            <origin xyz="${motor_h/2} 0 0" rpy="0 ${pi/2} 0"/>
             <mass value="${motor_m}" />
             <inertia    ixx="${1/12*motor_m*motor_h*motor_h+1/4*motor_m*motor_r*motor_r}" ixy="0" ixz="0" iyz="0"
@@ -217,5 +217,5 @@
     </link>
     <joint name="arm1_to_motor1" type="revolute">
-        <origin xyz="${arm_x-motor_r/2} 0 ${arm_z/2}" rpy="0 -1.57 0"/>
+        <origin xyz="${arm_x-motor_r} 0 ${arm_z/2}" rpy="0 -1.57 0"/>
         <parent link="arm1" />
         <child link="motor1" />
@@ -224,17 +224,17 @@
     <link name="motor2">
         <visual>
-        <origin xyz="${motor_r/2} 0 0" rpy="0 ${pi/2} 0"/>
-            <geometry>
-                <cylinder radius="${motor_r}" length="${motor_h}" />
-            </geometry>
-        </visual>
-        <collision>
-            <origin xyz="${motor_r/2} 0 0" rpy="0 ${pi/2} 0"/>
-            <geometry>
-                <cylinder radius="${motor_r}" length="${motor_h}" />
-            </geometry>
-        </collision>
-        <inertial>
-            <origin xyz="${motor_r/2} 0 0" rpy="0 ${pi/2} 0"/>
+        <origin xyz="${motor_h/2} 0 0" rpy="0 ${pi/2} 0"/>
+            <geometry>
+                <cylinder radius="${motor_r}" length="${motor_h}" />
+            </geometry>
+        </visual>
+        <collision>
+            <origin xyz="${motor_h/2} 0 0" rpy="0 ${pi/2} 0"/>
+            <geometry>
+                <cylinder radius="${motor_r}" length="${motor_h}" />
+            </geometry>
+        </collision>
+        <inertial>
+            <origin xyz="${motor_h/2} 0 0" rpy="0 ${pi/2} 0"/>
             <mass value="${motor_m}" />
             <inertia    ixx="${1/12*motor_m*motor_h*motor_h+1/4*motor_m*motor_r*motor_r}" ixy="0" ixz="0" iyz="0"
@@ -244,5 +244,5 @@
     </link>
     <joint name="arm2_to_motor2" type="revolute">
-        <origin xyz="${arm_x-motor_r/2} 0 ${arm_z/2}" rpy="0 -1.57 0"/>
+        <origin xyz="${arm_x-motor_r} 0 ${arm_z/2}" rpy="0 -1.57 0"/>
         <parent link="arm2" />
         <child link="motor2" />
@@ -251,17 +251,17 @@
     <link name="motor3">
         <visual>
-        <origin xyz="${motor_r/2} 0 0" rpy="0 ${pi/2} 0"/>
-            <geometry>
-                <cylinder radius="${motor_r}" length="${motor_h}" />
-            </geometry>
-        </visual>
-        <collision>
-            <origin xyz="${motor_r/2} 0 0" rpy="0 ${pi/2} 0"/>
-            <geometry>
-                <cylinder radius="${motor_r}" length="${motor_h}" />
-            </geometry>
-        </collision>
-        <inertial>
-            <origin xyz="${motor_r/2} 0 0" rpy="0 ${pi/2} 0"/>
+        <origin xyz="${motor_h/2} 0 0" rpy="0 ${pi/2} 0"/>
+            <geometry>
+                <cylinder radius="${motor_r}" length="${motor_h}" />
+            </geometry>
+        </visual>
+        <collision>
+            <origin xyz="${motor_h/2} 0 0" rpy="0 ${pi/2} 0"/>
+            <geometry>
+                <cylinder radius="${motor_r}" length="${motor_h}" />
+            </geometry>
+        </collision>
+        <inertial>
+            <origin xyz="${motor_h/2} 0 0" rpy="0 ${pi/2} 0"/>
             <mass value="${motor_m}" />
             <inertia    ixx="${1/12*motor_m*motor_h*motor_h+1/4*motor_m*motor_r*motor_r}" ixy="0" ixz="0" iyz="0"
@@ -271,5 +271,5 @@
     </link>
     <joint name="arm3_to_motor3" type="revolute">
-        <origin xyz="${arm_x-motor_r/2} 0 ${arm_z/2}" rpy="0 -1.57 0"/>
+        <origin xyz="${arm_x-motor_r} 0 ${arm_z/2}" rpy="0 -1.57 0"/>
         <parent link="arm3" />
         <child link="motor3" />
@@ -278,17 +278,17 @@
     <link name="motor4">
         <visual>
-        <origin xyz="${motor_r/2} 0 0" rpy="0 ${pi/2} 0"/>
-            <geometry>
-                <cylinder radius="${motor_r}" length="${motor_h}" />
-            </geometry>
-        </visual>
-        <collision>
-            <origin xyz="${motor_r/2} 0 0" rpy="0 ${pi/2} 0"/>
-            <geometry>
-                <cylinder radius="${motor_r}" length="${motor_h}" />
-            </geometry>
-        </collision>
-        <inertial>
-            <origin xyz="${motor_r/2} 0 0" rpy="0 ${pi/2} 0"/>
+        <origin xyz="${motor_h/2} 0 0" rpy="0 ${pi/2} 0"/>
+            <geometry>
+                <cylinder radius="${motor_r}" length="${motor_h}" />
+            </geometry>
+        </visual>
+        <collision>
+            <origin xyz="${motor_h/2} 0 0" rpy="0 ${pi/2} 0"/>
+            <geometry>
+                <cylinder radius="${motor_r}" length="${motor_h}" />
+            </geometry>
+        </collision>
+        <inertial>
+            <origin xyz="${motor_h/2} 0 0" rpy="0 ${pi/2} 0"/>
             <mass value="${motor_m}" />
             <inertia    ixx="${1/12*motor_m*motor_h*motor_h+1/4*motor_m*motor_r*motor_r}" ixy="0" ixz="0" iyz="0"
@@ -298,5 +298,5 @@
     </link>
     <joint name="arm4_to_motor4" type="revolute">
-        <origin xyz="${arm_x-motor_r/2} 0 ${arm_z/2}" rpy="0 -1.57 0"/>
+        <origin xyz="${arm_x-motor_r} 0 ${arm_z/2}" rpy="0 -1.57 0"/>
         <parent link="arm4" />
         <child link="motor4" />
@@ -305,17 +305,17 @@
          <link name="motor5">
         <visual>
-        <origin xyz="${motor_r/2} 0 0" rpy="0 ${pi/2} 0"/>
-            <geometry>
-                <cylinder radius="${motor_r}" length="${motor_h}" />
-            </geometry>
-        </visual>
-        <collision>
-            <origin xyz="${motor_r/2} 0 0" rpy="0 ${pi/2} 0"/>
-            <geometry>
-                <cylinder radius="${motor_r}" length="${motor_h}" />
-            </geometry>
-        </collision>
-        <inertial>
-            <origin xyz="${motor_r/2} 0 0" rpy="0 ${pi/2} 0"/>
+        <origin xyz="${motor_h/2} 0 0" rpy="0 ${pi/2} 0"/>
+            <geometry>
+                <cylinder radius="${motor_r}" length="${motor_h}" />
+            </geometry>
+        </visual>
+        <collision>
+            <origin xyz="${motor_h/2} 0 0" rpy="0 ${pi/2} 0"/>
+            <geometry>
+                <cylinder radius="${motor_r}" length="${motor_h}" />
+            </geometry>
+        </collision>
+        <inertial>
+            <origin xyz="${motor_h/2} 0 0" rpy="0 ${pi/2} 0"/>
             <mass value="${motor_m}" />
             <inertia    ixx="${1/12*motor_m*motor_h*motor_h+1/4*motor_m*motor_r*motor_r}" ixy="0" ixz="0" iyz="0"
@@ -325,5 +325,5 @@
     </link>
     <joint name="arm5_to_motor5" type="revolute">
-        <origin xyz="${arm_x-motor_r/2} 0 ${arm_z/2}" rpy="0 -1.57 0"/>
+        <origin xyz="${arm_x-motor_r} 0 ${arm_z/2}" rpy="0 -1.57 0"/>
         <parent link="arm5" />
         <child link="motor5" />
@@ -332,17 +332,17 @@
     <link name="motor6">
         <visual>
-        <origin xyz="${motor_r/2} 0 0" rpy="0 ${pi/2} 0"/>
-            <geometry>
-                <cylinder radius="${motor_r}" length="${motor_h}" />
-            </geometry>
-        </visual>
-        <collision>
-            <origin xyz="${motor_r/2} 0 0" rpy="0 ${pi/2} 0"/>
-            <geometry>
-                <cylinder radius="${motor_r}" length="${motor_h}" />
-            </geometry>
-        </collision>
-        <inertial>
-            <origin xyz="${motor_r/2} 0 0" rpy="0 ${pi/2} 0"/>
+        <origin xyz="${motor_h/2} 0 0" rpy="0 ${pi/2} 0"/>
+            <geometry>
+                <cylinder radius="${motor_r}" length="${motor_h}" />
+            </geometry>
+        </visual>
+        <collision>
+            <origin xyz="${motor_h/2} 0 0" rpy="0 ${pi/2} 0"/>
+            <geometry>
+                <cylinder radius="${motor_r}" length="${motor_h}" />
+            </geometry>
+        </collision>
+        <inertial>
+            <origin xyz="${motor_h/2} 0 0" rpy="0 ${pi/2} 0"/>
             <mass value="${motor_m}" />
             <inertia    ixx="${1/12*motor_m*motor_h*motor_h+1/4*motor_m*motor_r*motor_r}" ixy="0" ixz="0" iyz="0"
@@ -352,14 +352,14 @@
     </link>
     <joint name="arm6_to_motor6" type="revolute">
-        <origin xyz="${arm_x-motor_r/2} 0 ${arm_z/2}" rpy="0 -1.57 0"/>
+        <origin xyz="${arm_x-motor_r} 0 ${arm_z/2}" rpy="0 -1.57 0"/>
         <parent link="arm6" />
         <child link="motor6" />
         <limit effort="1000.0" velocity="0.5"/>  --default limits upper=lower=0
     </joint>
- -------------------------------------------------------------- axles
+ -------------------------------------------------------------------------------------------------- axles
 <!-- arm link -->
-<xacro:property name="axle_m" value="${body_m/20}" />
-<xacro:property name="axle_r" value="${body_s/40}" />
-<xacro:property name="axle_h" value="${body_s/40}" />
+<xacro:property name="axle_r" value="${0.003*body_s}" />
+<xacro:property name="axle_h" value="${0.001*body_s}" />
+<xacro:property name="axle_m" value="${0.001*body_m}" />
     <link name="axle1">
         <visual>
@@ -384,5 +384,5 @@
     </link>
     <joint name="motor1_to_axle1" type="continuous">
-        <origin xyz="${motor_r} 0 0" rpy="0 0 0"/>
+        <origin xyz="${motor_h+axle_h/2} 0 0" rpy="0 0 0"/>
         <axis xyz="1 0 0" />
         <parent link="motor1" />
@@ -411,5 +411,5 @@
     </link>
     <joint name="motor2_to_axle2" type="continuous">
-        <origin xyz="${motor_r} 0 0" rpy="0 0 0"/>
+        <origin xyz="${motor_h} 0 0" rpy="0 0 0"/>
         <axis xyz="1 0 0" />
         <parent link="motor2" />
@@ -438,5 +438,5 @@
     </link>
     <joint name="motor3_to_axle3" type="continuous">
-        <origin xyz="${motor_r} 0 0" rpy="0 0 0"/>
+        <origin xyz="${motor_h} 0 0" rpy="0 0 0"/>
         <axis xyz="1 0 0" />
         <parent link="motor3" />
@@ -465,5 +465,5 @@
     </link>
     <joint name="motor4_to_axle4" type="continuous">
-        <origin xyz="${motor_r} 0 0" rpy="0 0 0"/>
+        <origin xyz="${motor_h} 0 0" rpy="0 0 0"/>
         <axis xyz="1 0 0" />
         <parent link="motor4" />
@@ -492,5 +492,5 @@
     </link>
     <joint name="motor5_to_axle5" type="continuous">
-        <origin xyz="${motor_r} 0 0" rpy="0 0 0"/>
+        <origin xyz="${motor_h} 0 0" rpy="0 0 0"/>
         <axis xyz="1 0 0" />
         <parent link="motor5" />
@@ -519,30 +519,30 @@
     </link>
     <joint name="motor6_to_axle6" type="continuous">
-        <origin xyz="${motor_r} 0 0" rpy="0 0 0"/>
+        <origin xyz="${motor_h} 0 0" rpy="0 0 0"/>
         <axis xyz="1 0 0" />
         <parent link="motor6" />
         <child link="axle6" />
     </joint>
-  ------------------------------------------- propellers
+  ----------------------------------------------------------------------------------------------------- propellers
 <!-- propeller links -->
-<xacro:property name="propeller_m" value="${body_m/20}" />
-<xacro:property name="propeller_x" value="${1.5*body_s}" />
-<xacro:property name="propeller_y" value="${body_s/10}" />
-<xacro:property name="propeller_z" value="${body_s/40}" />
+<xacro:property name="propeller_x" value="${0.2*body_s}" />
+<xacro:property name="propeller_y" value="${0.015*body_s}" />
+<xacro:property name="propeller_z" value="${0.002*body_s}" />
+<xacro:property name="propeller_m" value="${0.001*body_m}" />
     <link name="prop1">
         <visual>
-            <origin xyz="0 0 0" rpy="0 ${pi/2} 0"/>
-            <geometry>
-                <box size="${propeller_x} ${propeller_y} ${propeller_z}" />
-            </geometry>
-        </visual>
-        <collision>
-            <origin xyz="0 0 0" rpy="0 ${pi/2} 0"/>
-            <geometry>
-                <box size="${propeller_x} ${propeller_y} ${propeller_z}" />
-            </geometry>
-        </collision>
-        <inertial>
-            <origin xyz="0 0 0" rpy="0 ${pi/2} 0"/>
+            <origin xyz="${propeller_z/2} 0 0" rpy="0 ${pi/2} 0"/>
+            <geometry>
+                <box size="${propeller_x} ${propeller_y} ${propeller_z}" />
+            </geometry>
+        </visual>
+        <collision>
+            <origin xyz="${propeller_z/2} 0 0" rpy="0 ${pi/2} 0"/>
+            <geometry>
+                <box size="${propeller_x} ${propeller_y} ${propeller_z}" />
+            </geometry>
+        </collision>
+        <inertial>
+            <origin xyz="${propeller_z/2} 0 0" rpy="0 ${pi/2} 0"/>
             <mass value="${propeller_m}" />
             <inertia    ixx="${1/12*propeller_m*(propeller_y*propeller_y+propeller_z*propeller_z)}" ixy="0" ixz="0" iyz="0"
@@ -559,17 +559,17 @@
     <link name="prop2">
         <visual>
-            <origin xyz="0 0 0" rpy="0 ${pi/2} 0"/>
-            <geometry>
-                <box size="${propeller_x} ${propeller_y} ${propeller_z}" />
-            </geometry>
-        </visual>
-        <collision>
-            <origin xyz="0 0 0" rpy="0 ${pi/2} 0"/>
-            <geometry>
-                <box size="${propeller_x} ${propeller_y} ${propeller_z}" />
-            </geometry>
-        </collision>
-        <inertial>
-            <origin xyz="0 0 0" rpy="0 ${pi/2} 0"/>
+            <origin xyz="${propeller_z/2} 0 0" rpy="0 ${pi/2} 0"/>
+            <geometry>
+                <box size="${propeller_x} ${propeller_y} ${propeller_z}" />
+            </geometry>
+        </visual>
+        <collision>
+            <origin xyz="${propeller_z/2} 0 0" rpy="0 ${pi/2} 0"/>
+            <geometry>
+                <box size="${propeller_x} ${propeller_y} ${propeller_z}" />
+            </geometry>
+        </collision>
+        <inertial>
+            <origin xyz="${propeller_z/2} 0 0" rpy="0 ${pi/2} 0"/>
             <mass value="${propeller_m}" />
             <inertia    ixx="${1/12*propeller_m*(propeller_y*propeller_y+propeller_z*propeller_z)}" ixy="0" ixz="0" iyz="0"
@@ -586,17 +586,17 @@
     <link name="prop3">
         <visual>
-            <origin xyz="0 0 0" rpy="0 ${pi/2} 0"/>
-            <geometry>
-                <box size="${propeller_x} ${propeller_y} ${propeller_z}" />
-            </geometry>
-        </visual>
-        <collision>
-            <origin xyz="0 0 0" rpy="0 ${pi/2} 0"/>
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
File: last_letter_2/config/param/models/plane_1wing/urdf/model.urdf.xacro (robot description, xacro)
@@ -97,5 +97,5 @@
         <child link="motor1" />
     </joint>
- -----------------------------------------------------------------------------------propeller
+ -------------------------------------------------------------------------------------------------- axle
 <!-- axle link parameters height, rad, mass-->
 <xacro:property name="axle_h" value="${0.02*body_s}" />
@@ -129,4 +129,5 @@
         <child link="axle1" />
     </joint>
+ -----------------------------------------------------------------------------------propeller
 <!-- propeller link parameters x, y, z, mass -->
 <xacro:property name="propeller_x" value="${0.26*body_s}" />

File: last_letter_2/config/param/models/plane_1wing_sensors/urdf/model.urdf.xacro (robot description, xacro)
@@ -97,5 +97,5 @@
       <child link="motor1" />
   </joint>
------------------------------------------------------------------------------------propeller
+-----------------------------------------------------------------------------------axle
 <!-- axle link parameters height, rad, mass-->
 <xacro:property name="axle_h" value="${0.02*body_s}" />
@@ -134,4 +134,5 @@
 <xacro:property name="propeller_z" value="${0.01*body_s}" />
 <xacro:property name="propeller_m" value="${0.015*mass}" />
+ -----------------------------------------------------------------------------------propeller
   <link name="prop1">
       <visual>

File: last_letter_2/config/param/models/plane_3wing_2motor/urdf/model.urdf.xacro (robot description, xacro)
@@ -183,5 +183,5 @@
         <child link="motor2" />
     </joint>
- -----------------------------------------------------------------------------------propeller
+ -----------------------------------------------------------------------------------axles
 <!-- axle link parameters height, rad, mass-->
 <xacro:property name="axle_h" value="${0.02*body_s}" />
@@ -242,4 +242,5 @@
         <child link="axle2" />
     </joint>
+ -----------------------------------------------------------------------------------propellers
 <!-- propeller link parameters x, y, z, mass -->
 <xacro:property name="propeller_x" value="${0.26*body_s}" />
