Commit message: copter controllers
Fix some details in multirotor's controller algorithm.

File: last_letter_2/config/param/models/quadcopter/urdf/model.urdf.xacro (robot description, xacro)
@@ -1,12 +1,12 @@
 <?xml version="1.0"?>
 <robot name="quadcopter" xmlns:xacro="http://www.ros.org/wiki/xacro">
-<xacro:property name="body_mass" value="1.5"/>
+<xacro:property name="body_mass" value="3"/>
 <!-- body, airfoil size -->
 <xacro:property name="body_s" value="1" />
 <!-- body link parameters x, y, z, mass-->
-<xacro:property name="body_x" value="${body_s}" />
-<xacro:property name="body_y" value="${body_s}" />
-<xacro:property name="body_z" value="${body_s/5}" />
-<xacro:property name="body_m" value="${body_mass}" />
+<xacro:property name="body_x" value="${0.1*body_s}" />
+<xacro:property name="body_y" value="${0.1*body_s}" />
+<xacro:property name="body_z" value="${0.02*body_s}" />
+<xacro:property name="body_m" value="${0.3*body_mass}" />
     <link name="body_FLU">
         <visual>
@@ -31,8 +31,8 @@
     </link>
 ---------------------------------------------------------- 4 quadcopter arms
-<xacro:property name="arm_x" value="${2*body_s}" />
-<xacro:property name="arm_y" value="${0.1*body_s}" />
-<xacro:property name="arm_z" value="${0.1*body_s}" />
-<xacro:property name="arm_m" value="${0.1*body_m}" />
+<xacro:property name="arm_x" value="${0.3*body_s}" />
+<xacro:property name="arm_y" value="${0.02*body_s}" />
+<xacro:property name="arm_z" value="${0.02*body_s}" />
+<xacro:property name="arm_m" value="${0.12*body_m}" />
     <link name="arm1">
         <visual>
@@ -140,8 +140,8 @@
     </joint>
     ------------------------------------------------------------------ motors
-<xacro:property name="motor_x" value="${0.2*body_s}" />
-<xacro:property name="motor_y" value="${0.2*body_s}" />
-<xacro:property name="motor_z" value="${0.2*body_s}" />
-<xacro:property name="motor_m" value="${0.1*body_m}" />
+<xacro:property name="motor_x" value="${0.01*body_s}" />
+<xacro:property name="motor_y" value="${0.02*body_s}" />
+<xacro:property name="motor_z" value="${0.02*body_s}" />
+<xacro:property name="motor_m" value="${0.05*body_m}" />
 <!-- only motor(Number_0f_Motor) acceptable name for motors -->
     <link name="motor1">
@@ -167,5 +167,5 @@
     </link>
     <joint name="arm1_to_motor1" type="revolute">
-        <origin xyz="${arm_x-motor_x/2} 0 ${arm_z/2}" rpy="0 -1.57 0"/>
+        <origin xyz="${arm_x-motor_z/2} 0 ${arm_z/2}" rpy="0 -1.57 0"/>
         <parent link="arm1" />
         <child link="motor1" />
@@ -194,5 +194,5 @@
     </link>
     <joint name="arm2_to_motor2" type="revolute">
-        <origin xyz="${arm_x-motor_x/2} 0 ${arm_z/2}" rpy="0 -1.57 0"/>
+        <origin xyz="${arm_x-motor_z/2} 0 ${arm_z/2}" rpy="0 -1.57 0"/>
         <parent link="arm2" />
         <child link="motor2" />
@@ -221,5 +221,5 @@
     </link>
     <joint name="arm3_to_motor3" type="revolute">
-        <origin xyz="${arm_x-motor_x/2} 0 ${arm_z/2}" rpy="0 -1.57 0"/>
+        <origin xyz="${arm_x-motor_z/2} 0 ${arm_z/2}" rpy="0 -1.57 0"/>
         <parent link="arm3" />
         <child link="motor3" />
@@ -248,14 +248,14 @@
     </link>
     <joint name="arm4_to_motor4" type="revolute">
-        <origin xyz="${arm_x-motor_x/2} 0 ${arm_z/2}" rpy="0 -1.57 0"/>
+        <origin xyz="${arm_x-motor_z/2} 0 ${arm_z/2}" rpy="0 -1.57 0"/>
         <parent link="arm4" />
         <child link="motor4" />
         <limit effort="1000.0" velocity="0.5"/>  --default limits upper=lower=0
     </joint>
- ------------------------------------------------------------------------------------- propellers
+ ------------------------------------------------------------------------------------- axles
 <!-- arm link -->
-<xacro:property name="axle_m" value="${body_m/20}" />
-<xacro:property name="axle_r" value="${body_s/40}" />
-<xacro:property name="axle_h" value="${body_s/40}" />
+<xacro:property name="axle_r" value="${0.002*body_s}" />
+<xacro:property name="axle_h" value="${0.003*body_s}" />
+<xacro:property name="axle_m" value="${0.001*body_m}" />
     <link name="axle1">
         <visual>
@@ -366,9 +366,10 @@
         <child link="axle4" />
     </joint>
+ ------------------------------------------------------------------------------------- propellers
 <!-- propeller links -->
-<xacro:property name="propeller_m" value="${body_m/20}" />
-<xacro:property name="propeller_x" value="${2*body_s}" />
-<xacro:property name="propeller_y" value="${body_s/10}" />
-<xacro:property name="propeller_z" value="${body_s/40}" />
+<xacro:property name="propeller_x" value="${0.3*body_s}" />
+<xacro:property name="propeller_y" value="${0.015*body_s}" />
+<xacro:property name="propeller_z" value="${0.002*body_s}" />
+<xacro:property name="propeller_m" value="${0.001*body_m}" />
     <link name="prop1">
         <visual>

File: last_letter_2/config/param/objects/can/urdf/can_model.urdf.xacro (robot description, xacro)
@@ -2,9 +2,9 @@
 <robot name="can" xmlns:xacro="http://www.ros.org/wiki/xacro">
 <!-- body, airfoil sizes -->
-<xacro:property name="body_s" value="0.1" />
+<xacro:property name="body_s" value="1" />
 <!-- body link parameters x, y, z, mass-->
-<xacro:property name="body_x" value="${body_s}" />
-<xacro:property name="body_y" value="${body_s}" />
-<xacro:property name="body_z" value="${body_s}" />
+<xacro:property name="body_x" value="${0.05*body_s}" />
+<xacro:property name="body_y" value="${0.05*body_s}" />
+<xacro:property name="body_z" value="${0.05*body_s}" />
 <xacro:property name="body_m" value="1" />
     <link name="base_link">

Commit message: copter controllers 2
fix some details

File: last_letter_2/config/param/models/hexacopter/urdf/model.urdf.xacro (robot description, xacro)
@@ -1,5 +1,5 @@
 <?xml version="1.0"?>
 <robot name="hexacopter" xmlns:xacro="http://www.ros.org/wiki/xacro">
-<xacro:property name="body_mass" value="3"/>
+<xacro:property name="body_mass" value="2"/>
 <!-- body, airfoil size -->
 <xacro:property name="body_s" value="1" />
@@ -526,5 +526,5 @@
   ----------------------------------------------------------------------------------------------------- propellers
 <!-- propeller links -->
-<xacro:property name="propeller_x" value="${0.2*body_s}" />
+<xacro:property name="propeller_x" value="${0.15*body_s}" />
 <xacro:property name="propeller_y" value="${0.015*body_s}" />
 <xacro:property name="propeller_z" value="${0.002*body_s}" />

File: last_letter_2/config/param/models/quadcopter/urdf/model.urdf.xacro (robot description, xacro)
@@ -1,5 +1,5 @@
 <?xml version="1.0"?>
 <robot name="quadcopter" xmlns:xacro="http://www.ros.org/wiki/xacro">
-<xacro:property name="body_mass" value="3"/>
+<xacro:property name="body_mass" value="2"/>
 <!-- body, airfoil size -->
 <xacro:property name="body_s" value="1" />
@@ -11,5 +11,4 @@
     <link name="body_FLU">
         <visual>
-        <origin rpy="0 0 0.785"/>
             <geometry>
                <box size="${body_x} ${body_y} ${body_z}" />
@@ -17,5 +16,4 @@
         </visual>
         <collision>
-        <origin rpy="0 0 0.785"/>
             <geometry>
                <box size="${body_x} ${body_y} ${body_z}" />
@@ -23,5 +21,4 @@
         </collision>
         <inertial>
-        <origin rpy="0 0 0.785"/>
             <mass value="${body_m}" />
              <inertia   ixx="${1/12*body_m*(body_y*body_y+body_z*body_z)}" ixy="0" ixz="0" iyz="0"
@@ -57,5 +54,5 @@
     </link>
     <joint name="body_FLU_to_arm1" type="fixed">
-        <origin xyz="${0.9*body_x/2} 0 0" rpy="0 0 0"/>
+        <origin xyz="0 0 0" rpy="0 0 ${7/4*pi}"/>
         <parent link="body_FLU" />
         <child link="arm1" />
@@ -83,5 +80,5 @@
     </link>
     <joint name="body_FLU_to_arm2" type="fixed">
-        <origin xyz="0 -${0.9*body_y/2} 0" rpy="0 0 ${3/2*pi}"/>
+        <origin xyz="0 0 0" rpy="0 0 ${5/4*pi}"/>
         <parent link="body_FLU" />
         <child link="arm2" />
@@ -109,5 +106,5 @@
     </link>
     <joint name="body_FLU_to_arm3" type="fixed">
-        <origin xyz="-${0.9*body_x/2} 0 0" rpy="0 0 ${pi}"/>
+        <origin xyz="0 0 0" rpy="0 0 ${3/4*pi}"/>
         <parent link="body_FLU" />
         <child link="arm3" />
@@ -135,5 +132,5 @@
     </link>
     <joint name="body_FLU_to_arm4" type="fixed">
-        <origin xyz="0 ${0.9*body_y/2} 0" rpy="0 0 ${1/2*pi}"/>
+        <origin xyz="0 0 0" rpy="0 0 ${1/4*pi}"/>
         <parent link="body_FLU" />
         <child link="arm4" />
@@ -368,5 +365,5 @@
  ------------------------------------------------------------------------------------- propellers
 <!-- propeller links -->
-<xacro:property name="propeller_x" value="${0.3*body_s}" />
+<xacro:property name="propeller_x" value="${0.15*body_s}" />
 <xacro:property name="propeller_y" value="${0.015*body_s}" />
 <xacro:property name="propeller_z" value="${0.002*body_s}" />
