Commit message: WIP: towards full PX4 SITL functionality
* Added IIR filter in acceleration measurement to avoid ground jitter
* Added euler2quat function in math_lib
* Fixed motor order and directions
* Fixed bug: magnetic reading is now in body frame
* Various rotation fixes
* Fixed bug in published coordinates ground truth

Still doesn't work correctly, orientation solution drifts, sensors pick biases.

File: last_letter_2/config/param/models/standard_vtol/urdf/model.urdf.xacro (robot description, xacro)
@@ -81,5 +81,5 @@
     </link>
     <joint name="body_FLU_to_arm2" type="fixed">
-        <origin xyz="0 0 0" rpy="0 0 ${5/4*pi}"/>
+        <origin xyz="0 0 0" rpy="0 0 ${3/4*pi}"/>
         <parent link="body_FLU" />
         <child link="arm2" />
@@ -107,5 +107,5 @@
     </link>
     <joint name="body_FLU_to_arm3" type="fixed">
-        <origin xyz="0 0 0" rpy="0 0 ${3/4*pi}"/>
+        <origin xyz="0 0 0" rpy="0 0 ${1/4*pi}"/>
         <parent link="body_FLU" />
         <child link="arm3" />
@@ -133,5 +133,5 @@
     </link>
     <joint name="body_FLU_to_arm4" type="fixed">
-        <origin xyz="0 0 0" rpy="0 0 ${1/4*pi}"/>
+        <origin xyz="0 0 0" rpy="0 0 ${5/4*pi}"/>
         <parent link="body_FLU" />
         <child link="arm4" />
